File: design/catsquirt_ioboard.sch (KiCad schematic (older format))
At the start: 6 parts

Commit message: Dan's style schema in KiCAD first uploaded
Parts:
- removed F?: 10A, symbol FUSE
- removed F?: 2A, symbol FUSE
- removed P?: BOSCH_MP5.2_37PIN, symbol BOSCH_MP5.2_37PIN
- removed P?: PA&PAD, symbol CONN_8X2_CATSQUIRT
- removed P?: IOC&PB, symbol CONN_8X2_CATSQUIRT
- removed P?: PP&Power, symbol CONN_8X2_CATSQUIRT
Connections:
- net labels added: AC_CLUTCH_RELAY, AC_SIGNAL, AN00, AN01, AN02, AN03, AN04, AN05, CHECK_ENGINE, CHT, EGO, FUEL_PUMP_RELAY, GAS_VENTI_VALVE, IAT, IGNITER_1_4, IGNITER_2_3, INJECTOR1-4, K_WIRE, L_WIRE, MAP, PA0, PA1, PA2, PA3, PA4, PA5, PA6, PA7, PB0, PB1, PB2, PB3, PP3, PP5, PP6, PP7, PT0, PT1, PT2, PT3, PT4, RFU_Injector_#1, RFU_Injector_#2, RFU_Injector_#3, RPM0+, RPM0-, RPM1+, RPM1-, RXD, SPEED_SENSOR, STEPPER_CLOSE, STEPPER_OPEN, TACH_OUT, TPS, TXD
- net labels removed: GND, com_rxd, com_txd, connector_1, connector_10, connector_11, connector_12, connector_13, connector_14, connector_15, connector_16, connector_17, connector_18, connector_19, connector_2, connector_20, connector_21, connector_22, connector_23, connector_24, connector_25, connector_26, connector_27, connector_28, connector_29, connector_3, connector_30, connector_31, connector_32, connector_33, connector_34, connector_35, connector_36, connector_37, connector_4, connector_5, connector_6, connector_7, connector_9, cpu_reg, shutdown
- wire segments 121 -> 109
- no-connect marks 22 -> 0
Other:
- note removed: "OEM ECU connector ripped\nfrom Bosch MP5.2"
