File: design/prototype.sch (KiCad schematic (older format))
At the start: 24 parts

Commit message: Ready to layout prototype board
Parts:
- added P4, P5: CONN_2, symbol CONN_2
- gave numbers to parts that had none: 24
Connections:
- net labels removed: AN00, AN01, AN02, AN03, AN05, PA0, PA1, PA2, PA3, PA4, PA5, PA6, PA7, PB0, PB1, PB2, PB3, PP3, PP5, PP6, PP7, PT1, PT2, PT3, RPM1+, RPM1-
- wire segments 69 -> 55
- no-connect marks 27 -> 51
Other:
- moved on the sheet: C1, C10, C11, C12, C2, C3, C4, C5, C6, C7, C8, C9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

Commit message: use sil-8 as board interface, arrange components on board
Parts:
- removed P1: PA&PAD, symbol CONN_8X2_CATSQUIRT
- removed P2: PP&Power, symbol CONN_8X2_CATSQUIRT
- removed P3: IOC&PB, symbol CONN_8X2_CATSQUIRT
- added P1: CONN_8, symbol CONN_8
Connections:
- no-connect marks 51 -> 17
Changed lines of the file:
@@
-EESchema Schematic File Version 2  date 21/10/2011 13:05:34
+EESchema Schematic File Version 2  date 25/10/2011 13:18:27
 LIBS:power
 LIBS:device
@@
 Sheet 1 1
 Title "prototype I/O board"
-Date "21 oct 2011"
+Date "25 oct 2011"
 Rev "0.01"
 Comp "diyefi.org"
@@
 Comment4 ""
 $EndDescr
-$Comp
-L +5V_MICRO #PWR01
-U 1 1 4EA0C960
-P 2950 1650
-F 0 "#PWR01" H 2950 1600 20  0001 C CNN
-F 1 "+5V_MICRO" H 2950 1750 30  0000 C CNN
-	1    2950 1650
-	1    0    0    -1
-$EndComp
+NoConn ~ 3900 1300
+NoConn ~ 3900 1200
+Wire Wire Line
+	4200 1950 4200 1900
+Wire Wire Line
+	4200 1900 3900 1900
 Connection ~ 6600 5700
 Wire Wire Line
@@
 	10450 5700 10450 5750
 Wire Wire Line
-	2950 1650 2950 1750
-Wire Wire Line
-	2950 1750 3150 1750
-Wire Wire Line
-	3150 1850 2950 1850
-Wire Wire Line
-	2950 1850 2950 1950
-Wire Wire Line
 	2050 5750 2050 5600
 Wire Wire Line
@@
 	6350 5300 8250 5300
 Connection ~ 6600 5300
+Wire Wire Line
+	3900 1800 4200 1800
+Wire Wire Line
+	4200 1800 4200 1700
+$Comp
+L CONN_8 P1
+U 1 1 4EA64596
+P 3550 1550
+F 0 "P1" V 3500 1550 60  0000 C CNN
+F 1 "CONN_8" V 3600 1550 60  0000 C CNN
+	1    3550 1550
+	-1   0    0    1
+$EndComp
+$Comp
+L PWR_FLAG #FLG01
+U 1 1 4EA4BE36
+P 6350 5500
+F 0 "#FLG01" H 6350 5770 30  0001 C CNN
+F 1 "PWR_FLAG" H 6350 5730 30  0000 C CNN
+	1    6350 5500
+	-1   0    0    1
+$EndComp
+$Comp
+L PWR_FLAG #FLG02
+U 1 1 4EA4BE0C
+P 6350 5300
+F 0 "#FLG02" H 6350 5570 30  0001 C CNN
+F 1 "PWR_FLAG" H 6350 5530 30  0000 C CNN
+	1    6350 5300
+	1    0    0    -1
+$EndComp
+NoConn ~ 9650 3750
+NoConn ~ 9650 3650
+NoConn ~ 9650 3550
+NoConn ~ 9650 3350
+NoConn ~ 9650 3150
+NoConn ~ 9650 3050
+$Comp
+L +5V_MICRO #PWR03
+U 1 1 4EA0C960
+P 4200 1700
+F 0 "#PWR03" H 4200 1650 20  0001 C CNN
+F 1 "+5V_MICRO" H 4200 1800 30  0000 C CNN
+	1    4200 1700
+	1    0    0    -1
+$EndComp
 $Comp
 L CONN_2 P4
@@
 $EndComp
 $Comp
-L +5V_SWITCHED #PWR02
+L +5V_SWITCHED #PWR04
 U 1 1 4E9FA4A2
 P 10050 5300
-F 0 "#PWR02" H 10050 5250 20  0001 C CNN
+F 0 "#PWR04" H 10050 5250 20  0001 C CNN
 F 1 "+5V_SWITCHED" H 10050 5400 30  0000 C CNN
 	1    10050 5300
 	1    0    0    -1
 $EndComp
-NoConn ~ 3950 1850
-NoConn ~ 3950 1750
-NoConn ~ 3950 1650
-NoConn ~ 3950 1450
 $Comp
 L CONN_2 P5
@@
 Text Label 1500 3600 2    60   ~ 0
 AN04
-Text Label 1950 1550 0    60   ~ 0
+Text Label 3900 1700 0    60   ~ 0
 AN04
-NoConn ~ 1150 1850
-NoConn ~ 1150 1750
-NoConn ~ 1150 1650
-NoConn ~ 1150 1550
-NoConn ~ 1150 1450
-NoConn ~ 1150 1350
-NoConn ~ 1150 1250
-NoConn ~ 1150 1150
-NoConn ~ 1950 1150
-NoConn ~ 1950 1250
-NoConn ~ 1950 1350
-NoConn ~ 1950 1450
-NoConn ~ 1950 1650
-NoConn ~ 5000 1250
-NoConn ~ 5000 1450
-NoConn ~ 5000 1350
-NoConn ~ 5800 1450
-NoConn ~ 5800 1350
-NoConn ~ 5800 1250
-NoConn ~ 5800 1150
-Text Label 5000 1150 2    60   ~ 0
+Text Label 3900 1600 0    60   ~ 0
 PT0
 Text Label 4650 5400 0    60   ~ 0
@@
 Text Label 7300 3250 2    60   ~ 0
 TXD
-Text Label 3150 1250 2    60   ~ 0
+Text Label 3900 1500 0    60   ~ 0
 RXD
-Text Label 3150 1150 2    60   ~ 0
+Text Label 3900 1400 0    60   ~ 0
 TXD
 $Comp
@@
 $EndComp
 $Comp
-L SENSORGND #PWR03
+L SENSORGND #PWR05
 U 1 1 4E9E51BF
 P 2750 6300
-F 0 "#PWR03" H 2750 6300 40  0001 C CNN
+F 0 "#PWR05" H 2750 6300 40  0001 C CNN
 F 1 "SENSORGND" H 2750 6230 40  0000 C CNN
 	1    2750 6300
@@
 $EndComp
 $Comp
-L +5V_SWITCHED #PWR04
+L +5V_SWITCHED #PWR06
 U 1 1 4E9E51BE
 P 4700 5700
-F 0 "#PWR04" H 4700 5650 20  0001 C CNN
+F 0 "#PWR06" H 4700 5650 20  0001 C CNN
 F 1 "+5V_SWITCHED" H 4700 5800 30  0000 C CNN
 	1    4700 5700
@@
 $EndComp
 $Comp
-L SENSORGND #PWR05
+L SENSORGND #PWR07
 U 1 1 4E9E51BD
 P 2050 5750
-F 0 "#PWR05" H 2050 5750 40  0001 C CNN
+F 0 "#PWR07" H 2050 5750 40  0001 C CNN
 F 1 "SENSORGND" H 2050 5680 40  0000 C CNN
 	1    2050 5750
@@
 $EndComp
 $Comp
-L CONN_8X2_CATSQUIRT P2
-U 1 1 4E9E51B3
-P 3550 1500
-F 0 "P2" H 3550 1950 60  0000 C CNN
-F 1 "PP&Power" V 3550 1500 50  0000 C CNN
-	1    3550 1500
-	-1   0    0    -1
-$EndComp
-$Comp
-L CONN_8X2_CATSQUIRT P3
-U 1 1 4E9E51B2
-P 5400 1500
-F 0 "P3" H 5400 1950 60  0000 C CNN
-F 1 "IOC&PB" V 5400 1500 50  0000 C CNN
-	1    5400 1500
-	1    0    0    -1
-$EndComp
-$Comp
-L CONN_8X2_CATSQUIRT P1
-U 1 1 4E9E51B1
-P 1550 1500
-F 0 "P1" H 1550 1950 60  0000 C CNN
-F 1 "PA&PAD" V 1550 1500 50  0000 C CNN
-	1    1550 1500
-	1    0    0    -1
-$EndComp
-NoConn ~ 1950 1750
-NoConn ~ 1950 1850
-NoConn ~ 5000 1550
-NoConn ~ 5000 1650
-NoConn ~ 5000 1750
-NoConn ~ 5000 1850
-NoConn ~ 5800 1550
-NoConn ~ 5800 1650
-NoConn ~ 5800 1750
-NoConn ~ 5800 1850
-$Comp
-L GND #PWR06
+L GND #PWR08
 U 1 1 4E9E51B0
-P 2950 1950
-F 0 "#PWR06" H 2950 1950 30  0001 C CNN
-F 1 "GND" H 2950 1880 30  0001 C CNN
-	1    2950 1950
-	1    0    0    -1
-$EndComp
-NoConn ~ 3150 1350
-NoConn ~ 3150 1450
-NoConn ~ 3150 1550
-NoConn ~ 3150 1650
-NoConn ~ 3950 1150
-NoConn ~ 3950 1250
-NoConn ~ 3950 1350
-NoConn ~ 3950 1550
-$Comp
-L SENSORGND #PWR07
+P 4200 1950
+F 0 "#PWR08" H 4200 1950 30  0001 C CNN
+F 1 "GND" H 4200 1880 30  0001 C CNN
+	1    4200 1950
+	1    0    0    -1
+$EndComp
+$Comp
+L SENSORGND #PWR09
 U 1 1 4E9E519A
 P 10450 5750
-F 0 "#PWR07" H 10450 5750 40  0001 C CNN
+F 0 "#PWR09" H 10450 5750 40  0001 C CNN
 F 1 "SENSORGND" H 10450 5680 40  0000 C CNN
 	1    10450 5750
@@
 $EndComp
 $Comp
-L GND #PWR08
+L GND #PWR010
 U 1 1 4E9E5198
 P 6600 5750
-F 0 "#PWR08" H 6600 5750 30  0001 C CNN
+F 0 "#PWR010" H 6600 5750 30  0001 C CNN
 F 1 "GND" H 6600 5680 30  0001 C CNN
 	1    6600 5750
@@
 $EndComp
 $Comp
-L +12V_SWITCHED #PWR09
+L +12V_SWITCHED #PWR011
 U 1 1 4E9E5193
 P 6600 5300
-F 0 "#PWR09" H 6600 5250 20  0001 C CNN
+F 0 "#PWR011" H 6600 5250 20  0001 C CNN
 F 1 "+12V_SWITCHED" H 6600 5400 30  0000 C CNN
 	1    6600 5300
@@
 $EndComp
 $Comp
-L +5V_MICRO #PWR010
+L +5V_MICRO #PWR012
 U 1 1 4E9E5192
 P 10450 5300
-F 0 "#PWR010" H 10450 5250 20  0001 C CNN
+F 0 "#PWR012" H 10450 5250 20  0001 C CNN
 F 1 "+5V_MICRO" H 10450 5400 30  0000 C CNN
 	1    10450 5300
@@
 $EndComp
 $Comp
-L GND #PWR011
+L GND #PWR013
 U 1 1 4E9E509E
 P 9750 2750
-F 0 "#PWR011" H 9750 2750 30  0001 C CNN
+F 0 "#PWR013" H 9750 2750 30  0001 C CNN
 F 1 "GND" H 9750 2680 30  0001 C CNN
 	1    9750 2750
@@
 $EndComp
 $Comp
-L +5V_SWITCHED #PWR012
+L +5V_SWITCHED #PWR014
 U 1 1 4E9E5098
 P 9400 2150
-F 0 "#PWR012" H 9400 2100 20  0001 C CNN
+F 0 "#PWR014" H 9400 2100 20  0001 C CNN
 F 1 "+5V_SWITCHED" H 9400 2250 30  0000 C CNN
 	1    9400 2150
@@
 $EndComp
 $Comp
-L GND #PWR013
+L GND #PWR015
 U 1 1 4E9E5096
 P 9500 3950
-F 0 "#PWR013" H 9500 3950 30  0001 C CNN
+F 0 "#PWR015" H 9500 3950 30  0001 C CNN
 F 1 "GND" H 9500 3880 30  0001 C CNN
 	1    9500 3950
@@
 $EndComp
 $Comp
-L +5V_SWITCHED #PWR014
+L +5V_SWITCHED #PWR016
 U 1 1 4E9E5082
 P 2550 2900
-F 0 "#PWR014" H 2550 2850 20  0001 C CNN
+F 0 "#PWR016" H 2550 2850 20  0001 C CNN
 F 1 "+5V_SWITCHED" H 2550 3000 30  0000 C CNN
 	1    2550 2900
@@
 $EndComp
 $Comp
-L SENSORGND #PWR015
+L SENSORGND #PWR017
 U 1 1 4E9E507E
 P 2250 4100
-F 0 "#PWR015" H 2250 4100 40  0001 C CNN
+F 0 "#PWR017" H 2250 4100 40  0001 C CNN
 F 1 "SENSORGND" H 2250 4030 40  0000 C CNN
 	1    2250 4100
