File: design/prototype.sch (KiCad schematic (older format))
At the start: 24 parts, among them J1 DB9, P1 CONN_8, P4 CONN_2, P5 CONN_2, U1 MAX232, U2 MPX4250A, U3 NCV1124, U4 TLE4275

Commit message: special design for toner transfer method, add serial monitor enable jumper
Parts:
- added JP1: JUMPER, symbol JUMPER
- added R5: 10K, symbol R
Connections:
- wire segments 55 -> 62
- no-connect marks 17 -> 16
Other:
- moved on the sheet: C1, C2, C3, C4, J1, U1
