File: design/Core Analogue Inputs.sch (KiCad schematic (older format))
At the start: 35 parts

Commit message: revise schema to be full pin compatible with stock ECU
Parts:
- gave numbers to parts that had none: 35
Connections:
- net labels added: ADCGND, AN06, GND
- net labels removed: AN05, SENSORGND
- wire segments 109 -> 78

Commit message: add test points on critical output, resolve all kind of DRC issue, generate a netlist
Parts:
- added W1: TEST, symbol TEST
Connections:
- wire segments 78 -> 81

Commit message: use max9924 to replace ncv1124, add narrow band oxygen sensor differential input circuit, put all component into PCB edge
Parts:
- added C46: 0.1u, symbol C
- added C47: 4.7u, symbol C
- added C48: 100P, symbol C
- added C49, C50, C51: 0.01u, symbol C
- added P4: CONN_2, symbol CONN_2
- added R72: 51.1K, symbol R
- added R73: 178K, symbol R
- added R74: 1K, symbol R
- added R75, R76: 4.22K, symbol R
- added U11: LM9040, symbol LM9040
Connections:
- net labels added: AN11, NBO2+, NBO2-
- net labels removed: EGO
- wire segments 81 -> 164
- no-connect marks 3 -> 6
Other:
- note added: "Wide band oxygen sensor"
- note added: "narrow band oxygen sensor"
- note removed: "Exhaust Gas Oxygen"
- moved on the sheet: C1, C10, C11, C12, C13, C2, C5, C6, C7, C8, C9, D1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

Commit message: make new footprint for max9924 & lm9040, add can bus interface, generate new netlist
Parts:
- P4: value CONN_2 -> WBO2
Connections:
- wire segments 164 -> 118
Other:
- note added: "Note 2"
- note added: "Note 2: The wideband O2 output should not share\n the stock harness, it should be soldered on board"
