File: design/Core Analogue Inputs.sch (KiCad schematic (older format))
At the start: 49 parts, among them K1 jumper, P4 WBO2, U1 MPX4250A, U11 LM9040

Commit message: revise schema according to Jaguar & Ravage project, eliminate as many errors as possible which were inherited from Puma board. Remove VSS interface, narrow band O2 interface, AC relay output, AC signal input. Make fuel injection configurable which can be batch fired or semi sequential fired
Parts:
- removed C46: 0.1u, symbol C
- removed C47: 4.7u, symbol C
- removed C48: 100P, symbol C
- removed C49, C50: 0.01u, symbol C
- removed K1: jumper, symbol CONN_3
- removed R72: 51.1K, symbol R
- removed R73: 178K, symbol R
- removed R74: 1K, symbol R
- removed R75, R76: 4.22K, symbol R
- removed U11: LM9040, symbol LM9040
- removed W1: TEST, symbol TEST
- C11: value 47pF -> 0.1uF
- C51: value 0.01u -> 0.33uF
- C9: value 0.1 -> 0.01uF
- R9: value 470R -> 1k
Connections:
- net labels removed: AN11, GND, MAP, NBO2+, NBO2-
- wire segments 118 -> 67
- no-connect marks 6 -> 3
Other:
- note added: "Note 1: The wideband O2 output should not share\n the stock harness, it should be screwed on board"
- note removed: "Note 1: Our MAP could be mounted externally\n through this jumper"
- note removed: "Note 2"
- note removed: "Note 2: The wideband O2 output should not share\n the stock harness, it should be soldered on board"
- note removed: "narrow band oxygen sensor"
- moved on the sheet: C1, C10, C11, C12, C13, C2, C3, C4, C5, C6, C7, C8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

Commit message: add hardware specs to README.md
Parts:
- D1, D10, D2, D3, D4, D5, D6, D7, D8, D9: value ZENER -> 1N5818-TP
Changed lines of the file:
@@
-EESchema Schematic File Version 2  date 02/02/2012 00:51:37
+EESchema Schematic File Version 2  date 02/02/2012 10:58:16
 LIBS:power
 LIBS:device
@@
 Sheet 5 10
 Title "Core Analogue Inputs"
-Date "1 feb 2012"
+Date "2 feb 2012"
 Rev "0.01"
 Comp "diyefi.org"
@@
 P 5500 5100
 F 0 "D10" H 5500 5200 50  0000 C CNN
-F 1 "ZENER" H 5500 5000 40  0000 C CNN
+F 1 "1N5818-TP" H 5500 5000 40  0000 C CNN
 	1    5500 5100
 	0    -1   -1   0
@@
 P 5500 4500
 F 0 "D9" H 5500 4600 50  0000 C CNN
-F 1 "ZENER" H 5500 4400 40  0000 C CNN
+F 1 "1N5818-TP" H 5500 4400 40  0000 C CNN
 	1    5500 4500
 	0    -1   -1   0
@@
 P 2000 4500
 F 0 "D7" H 2000 4600 50  0000 C CNN
-F 1 "ZENER" H 2000 4400 40  0000 C CNN
+F 1 "1N5818-TP" H 2000 4400 40  0000 C CNN
 	1    2000 4500
 	0    -1   -1   0
@@
 P 2000 5100
 F 0 "D8" H 2000 5200 50  0000 C CNN
-F 1 "ZENER" H 2000 5000 40  0000 C CNN
+F 1 "1N5818-TP" H 2000 5000 40  0000 C CNN
 	1    2000 5100
 	0    -1   -1   0
@@
 P 8650 2100
 F 0 "D3" H 8650 2200 50  0000 C CNN
-F 1 "ZENER" H 8650 2000 40  0000 C CNN
+F 1 "1N5818-TP" H 8650 2000 40  0000 C CNN
 	1    8650 2100
-	0    1    -1   0
+	0    -1   -1   0
 $EndComp
 $Comp
@@
 P 8650 2700
 F 0 "D6" H 8650 2800 50  0000 C CNN
-F 1 "ZENER" H 8650 2600 40  0000 C CNN
+F 1 "1N5818-TP" H 8650 2600 40  0000 C CNN
 	1    8650 2700
 	0    -1   -1   0
@@
 P 5450 2100
 F 0 "D2" H 5450 2200 50  0000 C CNN
-F 1 "ZENER" H 5450 2000 40  0000 C CNN
+F 1 "1N5818-TP" H 5450 2000 40  0000 C CNN
 	1    5450 2100
 	0    -1   -1   0
@@
 P 5450 2700
 F 0 "D5" H 5450 2800 50  0000 C CNN
-F 1 "ZENER" H 5450 2600 40  0000 C CNN
+F 1 "1N5818-TP" H 5450 2600 40  0000 C CNN
 	1    5450 2700
 	0    -1   -1   0
@@
 P 2000 2700
 F 0 "D4" H 2000 2800 50  0000 C CNN
-F 1 "ZENER" H 2000 2600 40  0000 C CNN
+F 1 "1N5818-TP" H 2000 2600 40  0000 C CNN
 	1    2000 2700
 	0    -1   -1   0
@@
 P 2000 2100
 F 0 "D1" H 2000 2200 50  0000 C CNN
-F 1 "ZENER" H 2000 2000 40  0000 C CNN
+F 1 "1N5818-TP" H 2000 2000 40  0000 C CNN
 	1    2000 2100
 	0    -1   -1   0

Commit message: make new footprint for screw connector, redesign ignition gnd & all lowside gnd
Parts:
- removed P4: WBO2, symbol CONN_2
Connections:
- net labels added: EGO
- wire segments 67 -> 65
Other:
- note removed: "Note 1"
- note removed: "Note 1: The wideband O2 output should not share\n the stock harness, it should be screwed on board"
- moved on the sheet: C3, C4, D2, D5, R4
Changed lines of the file:
@@
-EESchema Schematic File Version 2  date 02/02/2012 10:58:16
+EESchema Schematic File Version 2  date 07/02/2012 00:44:28
 LIBS:power
 LIBS:device
@@
 Sheet 5 10
 Title "Core Analogue Inputs"
-Date "2 feb 2012"
+Date "6 feb 2012"
 Rev "0.01"
 Comp "diyefi.org"
@@
 Comment4 ""
 $EndDescr
+Text HLabel 6400 2400 2    60   Input ~ 0
+EGO
 Connection ~ 8100 4400
 Wire Wire Line
@@
 	9050 4400 8700 4400
 Wire Wire Line
-	6050 2400 6500 2400
+	6100 2400 6400 2400
 Wire Wire Line
 	4950 5400 6200 5400
@@
 Wire Wire Line
 	9800 2400 9250 2400
-Connection ~ 4900 2400
-Wire Wire Line
-	5550 2400 4750 2400
-Wire Wire Line
-	5450 2900 5450 3100
-Wire Wire Line
-	6150 2900 6150 3000
-Wire Wire Line
-	4900 2900 4900 3000
-Wire Wire Line
-	5450 1900 5450 1700
-Wire Wire Line
-	5450 2300 5450 2500
-Connection ~ 5450 2400
-Wire Wire Line
-	4900 2500 4900 2400
-Connection ~ 5450 3000
+Connection ~ 4950 2400
+Wire Wire Line
+	5600 2400 4800 2400
+Wire Wire Line
+	5500 2900 5500 3100
+Wire Wire Line
+	6200 2900 6200 3000
+Wire Wire Line
+	4950 2900 4950 3000
+Wire Wire Line
+	5500 1900 5500 1700
+Wire Wire Line
+	5500 2300 5500 2500
+Connection ~ 5500 2400
+Wire Wire Line
+	4950 2500 4950 2400
+Connection ~ 5500 3000
 Wire Wire Line
 	2900 2400 2600 2400
@@
 Connection ~ 1450 2400
 Wire Wire Line
-	6150 2500 6150 2400
-Connection ~ 6150 2400
+	6200 2500 6200 2400
+Connection ~ 6200 2400
 Connection ~ 8100 2400
 Wire Wire Line
@@
 Connection ~ 6200 4800
 Wire Wire Line
-	4900 3000 6150 3000
+	4950 3000 6200 3000
 Wire Wire Line
 	1450 5400 2700 5400
-Wire Wire Line
-	6700 2400 6950 2400
-Wire Wire Line
-	6950 2400 6950 2700
 Wire Wire Line
 	2700 3000 1450 3000
@@
 $EndComp
 $Comp
-L ADCGND #PWR042
+L ADCGND #PWR046
 U 1 1 4F26B603
 P 7900 4900
-F 0 "#PWR042" H 7900 4900 40  0001 C CNN
+F 0 "#PWR046" H 7900 4900 40  0001 C CNN
 F 1 "ADCGND" H 7900 4830 40  0000 C CNN
 	1    7900 4900
@@
 $EndComp
 $Comp
-L ADCGND #PWR043
+L ADCGND #PWR047
 U 1 1 4F26A569
 P 8650 3100
-F 0 "#PWR043" H 8650 3100 40  0001 C CNN
+F 0 "#PWR047" H 8650 3100 40  0001 C CNN
 F 1 "ADCGND" H 8650 3030 40  0000 C CNN
 	1    8650 3100
 	1    0    0    -1
 $EndComp
-Text Notes 3900 7400 0    60   ~ 0
-Note 1: The wideband O2 output should not share\n the stock harness, it should be screwed on board
-Text Notes 6450 2300 0    60   ~ 0
-Note 1
-$Comp
-L ADCGND #PWR044
-U 1 1 4F19A01E
-P 6950 2700
-F 0 "#PWR044" H 6950 2700 40  0001 C CNN
-F 1 "ADCGND" H 6950 2630 40  0000 C CNN
-	1    6950 2700
-	1    0    0    -1
-$EndComp
-$Comp
-L CONN_2 P4
-U 1 1 4F199F3E
-P 6600 2750
-F 0 "P4" V 6550 2750 40  0000 C CNN
-F 1 "WBO2" V 6650 2750 40  0000 C CNN
-	1    6600 2750
-	0    -1   1    0
-$EndComp
-$Comp
-L ADCGND #PWR045
+$Comp
+L ADCGND #PWR048
 U 1 1 4EFDE581
 P 2000 5500
-F 0 "#PWR045" H 2000 5500 40  0001 C CNN
+F 0 "#PWR048" H 2000 5500 40  0001 C CNN
 F 1 "ADCGND" H 2000 5430 40  0000 C CNN
 	1    2000 5500
@@
 $EndComp
 $Comp
-L ADCGND #PWR046
+L ADCGND #PWR049
 U 1 1 4EFDE57C
 P 5500 5500
-F 0 "#PWR046" H 5500 5500 40  0001 C CNN
+F 0 "#PWR049" H 5500 5500 40  0001 C CNN
 F 1 "ADCGND" H 5500 5430 40  0000 C CNN
 	1    5500 5500
@@
 $EndComp
 $Comp
-L ADCGND #PWR047
+L ADCGND #PWR050
 U 1 1 4EFDE570
-P 5450 3100
-F 0 "#PWR047" H 5450 3100 40  0001 C CNN
-F 1 "ADCGND" H 5450 3030 40  0000 C CNN
-	1    5450 3100
-	1    0    0    -1
-$EndComp
-$Comp
-L ADCGND #PWR048
+P 5500 3100
+F 0 "#PWR050" H 5500 3100 40  0001 C CNN
+F 1 "ADCGND" H 5500 3030 40  0000 C CNN
+	1    5500 3100
+	1    0    0    -1
+$EndComp
+$Comp
+L ADCGND #PWR051
 U 1 1 4EFDE568
 P 2000 3100
-F 0 "#PWR048" H 2000 3100 40  0001 C CNN
+F 0 "#PWR051" H 2000 3100 40  0001 C CNN
 F 1 "ADCGND" H 2000 3030 40  0000 C CNN
 	1    2000 3100
@@
 $EndComp
 $Comp
-L +5V_SWITCHED #PWR049
+L +5V_SWITCHED #PWR052
 U 1 1 4E91936F
 P 7750 5150
-F 0 "#PWR049" H 7750 5100 20  0001 C CNN
+F 0 "#PWR052" H 7750 5100 20  0001 C CNN
 F 1 "+5V_SWITCHED" H 7750 5250 30  0000 C CNN
 	1    7750 5150
@@
 $EndComp
 $Comp
-L +5V_SWITCHED #PWR050
+L +5V_SWITCHED #PWR053
 U 1 1 4E91927A
 P 5500 4100
-F 0 "#PWR050" H 5500 4050 20  0001 C CNN
+F 0 "#PWR053" H 5500 4050 20  0001 C CNN
 F 1 "+5V_SWITCHED" H 5500 4200 30  0000 C CNN
 	1    5500 4100
@@
 $EndComp
 $Comp
-L +5V_SWITCHED #PWR051
+L +5V_SWITCHED #PWR054
 U 1 1 4E91916D
 P 2000 4100
-F 0 "#PWR051" H 2000 4050 20  0001 C CNN
+F 0 "#PWR054" H 2000 4050 20  0001 C CNN
 F 1 "+5V_SWITCHED" H 2000 4200 30  0000 C CNN
 	1    2000 4100
@@
 $EndComp
 $Comp
-L +12V_SWITCHED #PWR052
+L +12V_SWITCHED #PWR055
 U 1 1 4E919157
 P 9800 1700
-F 0 "#PWR052" H 9800 1650 20  0001 C CNN
+F 0 "#PWR055" H 9800 1650 20  0001 C CNN
 F 1 "+12V_SWITCHED" H 9800 1800 30  0000 C CNN
 	1    9800 1700
@@
 $EndComp
 $Comp
-L +5V_SWITCHED #PWR053
+L +5V_SWITCHED #PWR056
 U 1 1 4E919116
 P 8650 1700
-F 0 "#PWR053" H 8650 1650 20  0001 C CNN
+F 0 "#PWR056" H 8650 1650 20  0001 C CNN
 F 1 "+5V_SWITCHED" H 8650 1800 30  0000 C CNN
 	1    8650 1700
@@
 $EndComp
 $Comp
-L +5V_SWITCHED #PWR054
+L +5V_SWITCHED #PWR057
 U 1 1 4E9190CB
-P 5450 1700
-F 0 "#PWR054" H 5450 1650 20  0001 C CNN
-F 1 "+5V_SWITCHED" H 5450 1800 30  0000 C CNN
-	1    5450 1700
-	1    0    0    -1
-$EndComp
-$Comp
-L +5V_SWITCHED #PWR055
+P 5500 1700
+F 0 "#PWR057" H 5500 1650 20  0001 C CNN
+F 1 "+5V_SWITCHED" H 5500 1800 30  0000 C CNN
+	1    5500 1700
+	1    0    0    -1
+$EndComp
+$Comp
+L +5V_SWITCHED #PWR058
 U 1 1 4E9190BD
 P 2000 1700
-F 0 "#PWR055" H 2000 1650 20  0001 C CNN
+F 0 "#PWR058" H 2000 1650 20  0001 C CNN
 F 1 "+5V_SWITCHED" H 2000 1800 30  0000 C CNN
 	1    2000 1700
@@
 L ZENER D2
 U 1 1 4E918CA3
-P 5450 2100
-F 0 "D2" H 5450 2200 50  0000 C CNN
-F 1 "1N5818-TP" H 5450 2000 40  0000 C CNN
-	1    5450 2100
+P 5500 2100
+F 0 "D2" H 5500 2200 50  0000 C CNN
+F 1 "1N5818-TP" H 5500 2000 40  0000 C CNN
+	1    5500 2100
 	0    -1   -1   0
 $EndComp
@@
 L ZENER D5
 U 1 1 4E918CA2
-P 5450 2700
-F 0 "D5" H 5450 2800 50  0000 C CNN
-F 1 "1N5818-TP" H 5450 2600 40  0000 C CNN
-	1    5450 2700
+P 5500 2700
+F 0 "D5" H 5500 2800 50  0000 C CNN
+F 1 "1N5818-TP" H 5500 2600 40  0000 C CNN
+	1    5500 2700
 	0    -1   -1   0
 $EndComp
@@
 L R R4
 U 1 1 4E918CA1
-P 5800 2400
-F 0 "R4" V 5880 2400 50  0000 C CNN
-F 1 "470R" V 5800 2400 50  0000 C CNN
-	1    5800 2400
+P 5850 2400
+F 0 "R4" V 5930 2400 50  0000 C CNN
+F 1 "470R" V 5850 2400 50  0000 C CNN
+	1    5850 2400
 	0    1    1    0
 $EndComp
@@
 L C C3
 U 1 1 4E918C9F
-P 4900 2700
-F 0 "C3" H 4950 2800 50  0000 L CNN
-F 1 "0.22uF" H 4950 2600 50  0000 L CNN
-	1    4900 2700
+P 4950 2700
+F 0 "C3" H 5000 2800 50  0000 L CNN
+F 1 "0.22uF" H 5000 2600 50  0000 L CNN
+	1    4950 2700
 	1    0    0    -1
 $EndComp
@@
 L C C4
 U 1 1 4E918C9E
-P 6150 2700
-F 0 "C4" H 6200 2800 50  0000 L CNN
-F 1 "0.1uF" H 6200 2600 50  0000 L CNN
-	1    6150 2700
-	1    0    0    -1
-$EndComp
-Text HLabel 4750 2400 0    60   Output ~ 0
+P 6200 2700
+F 0 "C4" H 6250 2800 50  0000 L CNN
+F 1 "0.1uF" H 6250 2600 50  0000 L CNN
+	1    6200 2700
+	1    0    0    -1
+$EndComp
+Text HLabel 4800 2400 0    60   Output ~ 0
 AN03
-Text Notes 4950 3400 0    60   ~ 0
+Text Notes 5000 3400 0    60   ~ 0
 Wide band oxygen sensor
 Text Notes 1600 3400 0    60   ~ 0
