File: design/Low Side Drivers.sch (KiCad schematic (older format))
At the start: 25 parts

Commit message: revise schema to be full pin compatible with stock ECU
Parts:
- gave numbers to parts that had none: 25
Connections:
- net labels added: LSGND
- net labels removed: HCURGND
- wire segments 55 -> 45

Commit message: add test points on critical output, resolve all kind of DRC issue, generate a netlist
Parts:
- added W5: TEST, symbol TEST
Connections:
- wire segments 45 -> 48
Changed lines of the file:
@@
-EESchema Schematic File Version 2  date 02/01/2012 14:25:41
+EESchema Schematic File Version 2  date 03/01/2012 09:04:48
 LIBS:power
 LIBS:device
@@
 Sheet 7 12
 Title ""
-Date "2 jan 2012"
+Date "3 jan 2012"
 Rev ""
 Comp ""
@@
 $EndDescr
 Wire Wire Line
+	2600 6650 2600 6750
+Wire Wire Line
 	4450 6700 4450 6400
-$Comp
-L LSGND #PWR072
+Connection ~ 4450 5750
+Wire Wire Line
+	4450 6000 4450 5750
+Wire Wire Line
+	3650 5750 3800 5750
+Connection ~ 3300 6200
+Wire Wire Line
+	3950 6200 4150 6200
+Wire Wire Line
+	3050 6200 3450 6200
+Wire Wire Line
+	4750 5750 4200 5750
+Wire Wire Line
+	3150 5750 2800 5750
+Wire Wire Line
+	2800 5750 2800 5550
+Connection ~ 4450 3550
+Wire Wire Line
+	4450 3800 4450 3550
+Wire Wire Line
+	3650 3550 3800 3550
+Connection ~ 3300 4000
+Wire Wire Line
+	3300 4050 3300 4000
+Wire Wire Line
+	3950 4000 4150 4000
+Wire Wire Line
+	3050 4000 3450 4000
+Wire Wire Line
+	4450 4500 4450 4200
+Wire Wire Line
+	4750 3550 4200 3550
+Wire Wire Line
+	3150 3550 2800 3550
+Wire Wire Line
+	2800 3550 2800 3350
+Wire Wire Line
+	6100 3350 6100 3550
+Wire Wire Line
+	6100 3550 6450 3550
+Wire Wire Line
+	7500 3550 8050 3550
+Wire Wire Line
+	7750 4500 7750 4200
+Wire Wire Line
+	6750 4000 6350 4000
+Wire Wire Line
+	7250 4000 7450 4000
+Wire Wire Line
+	6600 4050 6600 4000
+Connection ~ 6600 4000
+Wire Wire Line
+	6950 3550 7100 3550
+Wire Wire Line
+	7750 3800 7750 3550
+Connection ~ 7750 3550
+Connection ~ 7750 1300
+Wire Wire Line
+	7750 1550 7750 1300
+Wire Wire Line
+	6950 1300 7100 1300
+Connection ~ 6600 1750
+Wire Wire Line
+	6600 1800 6600 1750
+Wire Wire Line
+	7250 1750 7450 1750
+Wire Wire Line
+	6350 1750 6750 1750
+Wire Wire Line
+	7750 2250 7750 1950
+Wire Wire Line
+	8050 1300 7500 1300
+Wire Wire Line
+	6450 1300 6100 1300
+Wire Wire Line
+	6100 1300 6100 1100
+Wire Wire Line
+	2800 1100 2800 1300
+Wire Wire Line
+	2800 1300 3150 1300
+Wire Wire Line
+	4200 1300 4750 1300
+Wire Wire Line
+	4450 2250 4450 1950
+Wire Wire Line
+	3450 1750 3050 1750
+Wire Wire Line
+	3950 1750 4150 1750
+Wire Wire Line
+	3300 1800 3300 1750
+Connection ~ 3300 1750
+Wire Wire Line
+	3650 1300 3800 1300
+Wire Wire Line
+	4450 1550 4450 1300
+Connection ~ 4450 1300
+Wire Wire Line
+	2600 6250 2600 6000
+Wire Wire Line
+	2600 6000 3300 6000
+Wire Wire Line
+	3300 6000 3300 6250
+$Comp
+L GND #PWR89
+U 1 1 4F025108
+P 2600 6750
+F 0 "#PWR89" H 2600 6750 30  0001 C CNN
+F 1 "GND" H 2600 6680 30  0001 C CNN
+	1    2600 6750
+	1    0    0    -1
+$EndComp
+$Comp
+L TEST W5
+U 1 1 4F0250C8
+P 2600 6450
+F 0 "W5" H 2600 6510 40  0000 C CNN
+F 1 "TEST" H 2600 6380 40  0000 C CNN
+	1    2600 6450
+	0    1    1    0
+$EndComp
+$Comp
+L LSGND #PWR88
 U 1 1 4EFDEDA3
 P 4450 6700
-F 0 "#PWR072" H 4450 6700 40  0001 C CNN
+F 0 "#PWR88" H 4450 6700 40  0001 C CNN
 F 1 "LSGND" H 4450 6630 40  0000 C CNN
 	1    4450 6700
@@
 $EndComp
 $Comp
-L LSGND #PWR073
+L LSGND #PWR84
 U 1 1 4EFDED9F
 P 7750 4500
-F 0 "#PWR073" H 7750 4500 40  0001 C CNN
+F 0 "#PWR84" H 7750 4500 40  0001 C CNN
 F 1 "LSGND" H 7750 4430 40  0000 C CNN
 	1    7750 4500
@@
 $EndComp
 $Comp
-L LSGND #PWR074
+L LSGND #PWR83
 U 1 1 4EFDED9A
 P 4450 4500
-F 0 "#PWR074" H 4450 4500 40  0001 C CNN
+F 0 "#PWR83" H 4450 4500 40  0001 C CNN
 F 1 "LSGND" H 4450 4430 40  0000 C CNN
 	1    4450 4500
@@
 $EndComp
 $Comp
-L LSGND #PWR075
+L LSGND #PWR78
 U 1 1 4EFDED95
 P 7750 2250
-F 0 "#PWR075" H 7750 2250 40  0001 C CNN
+F 0 "#PWR78" H 7750 2250 40  0001 C CNN
 F 1 "LSGND" H 7750 2180 40  0000 C CNN
 	1    7750 2250
@@
 $EndComp
 $Comp
-L LSGND #PWR076
+L LSGND #PWR77
 U 1 1 4EFDED8F
 P 4450 2250
-F 0 "#PWR076" H 4450 2250 40  0001 C CNN
+F 0 "#PWR77" H 4450 2250 40  0001 C CNN
 F 1 "LSGND" H 4450 2180 40  0000 C CNN
 	1    4450 2250
@@
 $EndComp
 $Comp
-L +12V_SWITCHED #PWR077
+L +12V_SWITCHED #PWR87
 U 1 1 4E927233
 P 2800 5550
-F 0 "#PWR077" H 2800 5500 20  0001 C CNN
+F 0 "#PWR87" H 2800 5500 20  0001 C CNN
 F 1 "+12V_SWITCHED" H 2800 5650 30  0000 C CNN
 	1    2800 5550
 	1    0    0    -1
 $EndComp
-Connection ~ 4450 5750
-Wire Wire Line
-	4450 6000 4450 5750
-Wire Wire Line
-	3650 5750 3800 5750
-Connection ~ 3300 6200
-Wire Wire Line
-	3300 6250 3300 6200
-Wire Wire Line
-	3950 6200 4150 6200
-Wire Wire Line
-	3050 6200 3450 6200
-Wire Wire Line
-	4750 5750 4200 5750
-Wire Wire Line
-	3150 5750 2800 5750
-Wire Wire Line
-	2800 5750 2800 5550
 $Comp
 L R R53
@@
 $EndComp
 $Comp
-L GND #PWR078
+L GND #PWR90
 U 1 1 4E927230
 P 3300 6750
-F 0 "#PWR078" H 3300 6750 30  0001 C CNN
+F 0 "#PWR90" H 3300 6750 30  0001 C CNN
 F 1 "GND" H 3300 6680 30  0001 C CNN
 	1    3300 6750
@@
 Fuel Pump Relay Driver
 $Comp
-L +12V_SWITCHED #PWR079
+L +12V_SWITCHED #PWR81
 U 1 1 4E924B5B
 P 2800 3350
-F 0 "#PWR079" H 2800 3300 20  0001 C CNN
+F 0 "#PWR81" H 2800 3300 20  0001 C CNN
 F 1 "+12V_SWITCHED" H 2800 3450 30  0000 C CNN
 	1    2800 3350
 	1    0    0    -1
 $EndComp
-Connection ~ 4450 3550
-Wire Wire Line
-	4450 3800 4450 3550
-Wire Wire Line
-	3650 3550 3800 3550
-Connection ~ 3300 4000
-Wire Wire Line
-	3300 4050 3300 4000
-Wire Wire Line
-	3950 4000 4150 4000
-Wire Wire Line
-	3050 4000 3450 4000
-Wire Wire Line
-	4450 4500 4450 4200
-Wire Wire Line
-	4750 3550 4200 3550
-Wire Wire Line
-	3150 3550 2800 3550
-Wire Wire Line
-	2800 3550 2800 3350
 $Comp
 L R R47
@@
 $EndComp
 $Comp
-L GND #PWR080
+L GND #PWR85
 U 1 1 4E924B58
 P 3300 4550
-F 0 "#PWR080" H 3300 4550 30  0001 C CNN
+F 0 "#PWR85" H 3300 4550 30  0001 C CNN
 F 1 "GND" H 3300 4480 30  0001 C CNN
 	1    3300 4550
@@
 $EndComp
 $Comp
-L GND #PWR081
+L GND #PWR86
 U 1 1 4E924B22
 P 6600 4550
-F 0 "#PWR081" H 6600 4550 30  0001 C CNN
+F 0 "#PWR86" H 6600 4550 30  0001 C CNN
 F 1 "GND" H 6600 4480 30  0001 C CNN
 	1    6600 4550
@@
 	0    1    1    0
 $EndComp
-Wire Wire Line
-	6100 3350 6100 3550
-Wire Wire Line
-	6100 3550 6450 3550
-Wire Wire Line
-	7500 3550 8050 3550
-Wire Wire Line
-	7750 4500 7750 4200
-Wire Wire Line
-	6750 4000 6350 4000
-Wire Wire Line
-	7250 4000 7450 4000
-Wire Wire Line
-	6600 4050 6600 4000
-Connection ~ 6600 4000
-Wire Wire Line
-	6950 3550 7100 3550
-Wire Wire Line
-	7750 3800 7750 3550
-Connection ~ 7750 3550
-$Comp
-L +12V_SWITCHED #PWR082
+$Comp
+L +12V_SWITCHED #PWR82
 U 1 1 4E924B1F
 P 6100 3350
-F 0 "#PWR082" H 6100 3300 20  0001 C CNN
+F 0 "#PWR82" H 6100 3300 20  0001 C CNN
 F 1 "+12V_SWITCHED" H 6100 3450 30  0000 C CNN
 	1    6100 3350
@@
 $EndComp
 $Comp
-L +12V_SWITCHED #PWR083
+L +12V_SWITCHED #PWR76
 U 1 1 4E924B0C
 P 6100 1100
-F 0 "#PWR083" H 6100 1050 20  0001 C CNN
+F 0 "#PWR76" H 6100 1050 20  0001 C CNN
 F 1 "+12V_SWITCHED" H 6100 1200 30  0000 C CNN
 	1    6100 1100
@@
 $EndComp
 $Comp
-L +12V_SWITCHED #PWR084
+L +12V_SWITCHED #PWR75
 U 1 1 4E924B04
 P 2800 1100
-F 0 "#PWR084" H 2800 1050 20  0001 C CNN
+F 0 "#PWR75" H 2800 1050 20  0001 C CNN
 F 1 "+12V_SWITCHED" H 2800 1200 30  0000 C CNN
 	1    2800 1100
 	1    0    0    -1
 $EndComp
-Connection ~ 7750 1300
-Wire Wire Line
-	7750 1550 7750 1300
-Wire Wire Line
-	6950 1300 7100 1300
-Connection ~ 6600 1750
-Wire Wire Line
-	6600 1800 6600 1750
-Wire Wire Line
-	7250 1750 7450 1750
-Wire Wire Line
-	6350 1750 6750 1750
-Wire Wire Line
-	7750 2250 7750 1950
-Wire Wire Line
-	8050 1300 7500 1300
-Wire Wire Line
-	6450 1300 6100 1300
-Wire Wire Line
-	6100 1300 6100 1100
 $Comp
 L R R42
@@
 $EndComp
 $Comp
-L GND #PWR085
+L GND #PWR80
 U 1 1 4E924A81
 P 6600 2300
-F 0 "#PWR085" H 6600 2300 30  0001 C CNN
+F 0 "#PWR80" H 6600 2300 30  0001 C CNN
 F 1 "GND" H 6600 2230 30  0001 C CNN
 	1    6600 2300
@@
 $EndComp
 $Comp
-L GND #PWR086
+L GND #PWR79
 U 1 1 4E919D92
 P 3300 2300
-F 0 "#PWR086" H 3300 2300 30  0001 C CNN
+F 0 "#PWR79" H 3300 2300 30  0001 C CNN
 F 1 "GND" H 3300 2230 30  0001 C CNN
 	1    3300 2300
@@
 	0    1    1    0
 $EndComp
-Wire Wire Line
-	2800 1100 2800 1300
-Wire Wire Line
-	2800 1300 3150 1300
-Wire Wire Line
-	4200 1300 4750 1300
-Wire Wire Line
-	4450 2250 4450 1950
-Wire Wire Line
-	3450 1750 3050 1750
-Wire Wire Line
-	3950 1750 4150 1750
-Wire Wire Line
-	3300 1800 3300 1750
-Connection ~ 3300 1750
-Wire Wire Line
-	3650 1300 3800 1300
-Wire Wire Line
-	4450 1550 4450 1300
-Connection ~ 4450 1300
 $EndSCHEMATC

Commit message: add missing diodes, re-generate netlist, assign all footprints, ready to layout
Parts:
- added D19, D20, D23, D24, D26: DIODE, symbol DIODE
- renumbered D16 to D17, D17 to D18, D18 to D21, D19 to D22, D20 to D25
Connections:
- wire segments 48 -> 58
Changed lines of the file:
@@
-EESchema Schematic File Version 2  date 03/01/2012 09:04:48
+EESchema Schematic File Version 2  date 12/01/2012 20:05:35
 LIBS:power
 LIBS:device
@@
 $Descr A4 11700 8267
 Sheet 7 12
-Title ""
-Date "3 jan 2012"
-Rev ""
-Comp ""
+Title "low side drivers"
+Date "12 jan 2012"
+Rev "0.01"
+Comp "diyefi.org"
 Comment1 ""
 Comment2 ""
@@
 $EndDescr
 Wire Wire Line
+	4700 6400 4450 6400
+Wire Wire Line
+	8000 4200 7750 4200
+Wire Wire Line
+	4700 4200 4450 4200
+Wire Wire Line
+	8000 1950 7750 1950
+Wire Wire Line
+	4700 1950 4450 1950
+Wire Wire Line
 	2600 6650 2600 6750
 Wire Wire Line
-	4450 6700 4450 6400
+	4450 6400 4450 6700
 Connection ~ 4450 5750
 Wire Wire Line
-	4450 6000 4450 5750
+	4450 5750 4450 6000
 Wire Wire Line
 	3650 5750 3800 5750
@@
 Connection ~ 4450 3550
 Wire Wire Line
-	4450 3800 4450 3550
+	4450 3550 4450 3800
 Wire Wire Line
 	3650 3550 3800 3550
@@
 	3050 4000 3450 4000
 Wire Wire Line
-	4450 4500 4450 4200
+	4450 4200 4450 4500
 Wire Wire Line
 	4750 3550 4200 3550
@@
 	7500 3550 8050 3550
 Wire Wire Line
-	7750 4500 7750 4200
+	7750 4200 7750 4500
 Wire Wire Line
 	6750 4000 6350 4000
@@
 	6950 3550 7100 3550
 Wire Wire Line
-	7750 3800 7750 3550
+	7750 3550 7750 3800
 Connection ~ 7750 3550
 Connection ~ 7750 1300
 Wire Wire Line
-	7750 1550 7750 1300
+	7750 1300 7750 1550
 Wire Wire Line
 	6950 1300 7100 1300
@@
 	6350 1750 6750 1750
 Wire Wire Line
-	7750 2250 7750 1950
+	7750 1950 7750 2250
 Wire Wire Line
 	8050 1300 7500 1300
@@
 	4200 1300 4750 1300
 Wire Wire Line
-	4450 2250 4450 1950
+	4450 1950 4450 2250
 Wire Wire Line
 	3450 1750 3050 1750
@@
 	3650 1300 3800 1300
 Wire Wire Line
-	4450 1550 4450 1300
+	4450 1300 4450 1550
 Connection ~ 4450 1300
 Wire Wire Line
@@
 Wire Wire Line
 	3300 6000 3300 6250
+Wire Wire Line
+	4450 1550 4700 1550
+Wire Wire Line
+	7750 1550 8000 1550
+Wire Wire Line
+	4450 3800 4700 3800
+Wire Wire Line
+	7750 3800 8000 3800
+Wire Wire Line
+	4450 6000 4700 6000
+$Comp
+L DIODE D26
+U 1 1 4F0ECBC1
+P 4700 6200
+F 0 "D26" H 4700 6300 40  0000 C CNN
+F 1 "DIODE" H 4700 6100 40  0000 C CNN
+	1    4700 6200
+	0    -1   -1   0
+$EndComp
+$Comp
+L DIODE D24
+U 1 1 4F0ECBB4
+P 8000 4000
+F 0 "D24" H 8000 4100 40  0000 C CNN
+F 1 "DIODE" H 8000 3900 40  0000 C CNN
+	1    8000 4000
+	0    -1   -1   0
+$EndComp
+$Comp
+L DIODE D23
+U 1 1 4F0ECBA9
+P 4700 4000
+F 0 "D23" H 4700 4100 40  0000 C CNN
+F 1 "DIODE" H 4700 3900 40  0000 C CNN
+	1    4700 4000
+	0    -1   -1   0
+$EndComp
+$Comp
+L DIODE D20
+U 1 1 4F0ECB9C
+P 8000 1750
+F 0 "D20" H 8000 1850 40  0000 C CNN
+F 1 "DIODE" H 8000 1650 40  0000 C CNN
+	1    8000 1750
+	0    -1   -1   0
+$EndComp
+$Comp
+L DIODE D19
+U 1 1 4F0ECB85
+P 4700 1750
+F 0 "D19" H 4700 1850 40  0000 C CNN
+F 1 "DIODE" H 4700 1650 40  0000 C CNN
+	1    4700 1750
+	0    -1   -1   0
+$EndComp
 $Comp
 L GND #PWR89
@@
 $EndComp
 $Comp
-L LED D20
+L LED D25
 U 1 1 4E927231
 P 4000 5750
-F 0 "D20" H 4000 5850 50  0000 C CNN
+F 0 "D25" H 4000 5850 50  0000 C CNN
 F 1 "LED" H 4000 5650 50  0000 C CNN
 	1    4000 5750
@@
 $EndComp
 $Comp
-L LED D18
+L LED D21
 U 1 1 4E924B59
 P 4000 3550
-F 0 "D18" H 4000 3650 50  0000 C CNN
+F 0 "D21" H 4000 3650 50  0000 C CNN
 F 1 "LED" H 4000 3450 50  0000 C CNN
 	1    4000 3550
@@
 $EndComp
 $Comp
-L LED D19
+L LED D22
 U 1 1 4E924B21
 P 7300 3550
-F 0 "D19" H 7300 3650 50  0000 C CNN
+F 0 "D22" H 7300 3650 50  0000 C CNN
 F 1 "LED" H 7300 3450 50  0000 C CNN
 	1    7300 3550
@@
 $EndComp
 $Comp
-L LED D17
+L LED D18
 U 1 1 4E924A82
 P 7300 1300
-F 0 "D17" H 7300 1400 50  0000 C CNN
+F 0 "D18" H 7300 1400 50  0000 C CNN
 F 1 "LED" H 7300 1200 50  0000 C CNN
 	1    7300 1300
@@
 $EndComp
 $Comp
-L LED D16
+L LED D17
 U 1 1 4E919D91
 P 4000 1300
-F 0 "D16" H 4000 1400 50  0000 C CNN
+F 0 "D17" H 4000 1400 50  0000 C CNN
 F 1 "LED" H 4000 1200 50  0000 C CNN
 	1    4000 1300
