File: design/Low Side Drivers.sch (KiCad schematic (older format))
At the start: 31 parts, among them Q4 vnp10n07, Q5 vnp10n07, Q6 vnp10n07, Q7 vnp10n07, Q8 vnp10n07

Commit message: revise schema according to Jaguar & Ravage project, eliminate as many errors as possible which were inherited from Puma board. Remove VSS interface, narrow band O2 interface, AC relay output, AC signal input. Make fuel injection configurable which can be batch fired or semi sequential fired
Parts:
- removed D18: LED, symbol LED
- removed D19: DIODE, symbol DIODE
- removed Q5: vnp10n07, symbol MOS_N
- removed R42: 2K4, symbol R
- removed R44: 1K, symbol R
- removed R46: 100K, symbol R
- removed W5: TEST, symbol TEST
- D20, D23, D24, D26: value DIODE -> 1N4148
Connections:
- net labels removed: AC_CLUTCH_RELAY, PP5
- wire segments 58 -> 36
Other:
- note removed: "AC compressor clutch relay"
- moved on the sheet: D17, D21, D22, D25, Q4, Q6, Q7, Q8, R41, R43, R45, R47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
