File: design/Power Supplies.sch (KiCad schematic (older format))
At the start: 15 parts

Commit message: revise schema to be full pin compatible with stock ECU
Parts:
- gave numbers to parts that had none: 15
Connections:
- net labels added: ADCGND, IGNGND, LSGND
- net labels removed: HCURGND, SENSORGND
- wire segments 42 -> 20
Other:
- note added: "Power symbols\n+12V_SWITCHED come from igniton switch\n+5V_MICRO come from CPU voltage reg \n+5V_SWITCHED come from secondary voltage reg\nLSGND low side ground\nADCGND sensor ground\nIGNGND ignition ground"
- moved on the sheet: C39, C40, C41, C42, C43, C44, C45, C46, C47, C48, C49, C50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

Commit message: add test points on critical output, resolve all kind of DRC issue, generate a netlist
Parts:
- removed C43, C44: 10uF, C1V7, symbol CAPAPOL
- removed C45, C46: .1uF, C1V7, symbol C
- removed C47, C48: 22uF, symbol C
- removed C49: 2200uF, C1V7, symbol CAPAPOL
- removed C50: 0.001uF, symbol C
- removed U10: LM9076Q, symbol LM9076Q
- added C43: 22uF, symbol C
- added C44: 470nF, symbol C
- added R70: 29K4, symbol R
- added R71: 10K, symbol R
- added U10: LM2941S, symbol LM2941S
- R69: value 10K -> 33K
Connections:
- wire segments 20 -> 26
- no-connect marks 0 -> 1

Commit message: some fixes on pin layout to pass footprint tests, did a manual modules placement, get all holes sit on right place
Connections:
- wire segments 26 -> 27
- no-connect marks 1 -> 0
Changed lines of the file:
@@
-EESchema Schematic File Version 2  date 12/01/2012 20:05:35
+EESchema Schematic File Version 2  date 14/01/2012 13:46:11
 LIBS:power
 LIBS:device
@@
 Sheet 12 12
 Title "Power supplies"
-Date "12 jan 2012"
+Date "14 jan 2012"
 Rev "0.01"
 Comp "diyefi.org"
@@
 Comment4 ""
 $EndDescr
+Connection ~ 5350 4900
+Wire Wire Line
+	5350 4400 5350 4900
+Connection ~ 7100 4900
+Wire Wire Line
+	7100 5000 7100 4900
+Wire Wire Line
+	6600 4400 6600 5000
+Connection ~ 6850 4900
+Wire Wire Line
+	7600 4500 7600 4900
+Wire Wire Line
+	7600 4900 4450 4900
+Wire Wire Line
+	7100 4400 6850 4400
+Wire Wire Line
+	7100 4400 7100 4750
+Wire Wire Line
+	7100 4750 7300 4750
+Wire Wire Line
+	7300 4250 7300 4100
+Wire Wire Line
+	4450 4900 4450 4700
+Wire Wire Line
+	4250 5200 4800 5200
+Wire Wire Line
+	4800 5200 4800 4750
+Connection ~ 4800 4100
+Wire Wire Line
+	4800 4100 4800 4250
+Wire Wire Line
+	5900 2700 5900 2900
+Wire Wire Line
+	7200 2800 4700 2800
+Connection ~ 5100 2400
+Connection ~ 5100 2800
+Connection ~ 7200 2400
+Connection ~ 6750 2800
+Connection ~ 4700 2400
+Connection ~ 4700 2800
+Connection ~ 6750 2400
+Wire Wire Line
+	4300 2400 5500 2400
+Connection ~ 5900 2800
+Wire Wire Line
+	7600 2400 6300 2400
+Connection ~ 5900 2800
+Connection ~ 6750 2400
+Connection ~ 4700 2800
+Connection ~ 4700 2400
+Connection ~ 6750 2800
+Connection ~ 7200 2400
+Connection ~ 5100 2800
+Connection ~ 5100 2400
+Connection ~ 7200 2800
+Wire Wire Line
+	5350 4100 4050 4100
+Wire Wire Line
+	4450 4100 4450 4300
+Connection ~ 4450 4100
+Wire Wire Line
+	4800 4750 5150 4750
+Connection ~ 4800 4750
+Wire Wire Line
+	5150 4750 5150 4250
+Wire Wire Line
+	5150 4250 5350 4250
+Connection ~ 6600 4900
+Wire Wire Line
+	6600 4250 6850 4250
+Wire Wire Line
+	6850 4250 6850 4400
+Connection ~ 7300 4100
+Wire Wire Line
+	8000 4100 6600 4100
+Connection ~ 7600 4100
+Wire Wire Line
+	6850 5000 6850 4900
+Wire Wire Line
+	7350 5000 7350 4900
+Connection ~ 7350 4900
 $Comp
 L PWR_FLAG #FLG3
@@
 	1    0    0    -1
 $EndComp
-Connection ~ 7350 4900
-Wire Wire Line
-	7350 5000 7350 4900
-Wire Wire Line
-	6850 5000 6850 4900
-Connection ~ 7600 4100
-Wire Wire Line
-	8000 4100 6600 4100
-Connection ~ 7300 4100
-Wire Wire Line
-	6850 4250 6850 4400
-Wire Wire Line
-	6850 4250 6600 4250
-Connection ~ 6600 4900
-Wire Wire Line
-	5350 4250 5150 4250
-Wire Wire Line
-	5150 4250 5150 4750
-Connection ~ 4800 4750
-Wire Wire Line
-	5150 4750 4800 4750
-Connection ~ 4450 4100
-Wire Wire Line
-	4450 4100 4450 4300
-Wire Wire Line
-	5350 4100 4050 4100
-Connection ~ 7200 2800
-Connection ~ 5100 2400
-Connection ~ 5100 2800
-Connection ~ 7200 2400
-Connection ~ 6750 2800
-Connection ~ 4700 2400
-Connection ~ 4700 2800
-Connection ~ 6750 2400
-Connection ~ 5900 2800
-Wire Wire Line
-	7600 2400 6300 2400
-Connection ~ 5900 2800
-Wire Wire Line
-	4300 2400 5500 2400
-Connection ~ 6750 2400
-Connection ~ 4700 2800
-Connection ~ 4700 2400
-Connection ~ 6750 2800
-Connection ~ 7200 2400
-Connection ~ 5100 2800
-Connection ~ 5100 2400
-Wire Wire Line
-	7200 2800 4700 2800
-Wire Wire Line
-	5900 2700 5900 2900
-Wire Wire Line
-	4800 4100 4800 4250
-Connection ~ 4800 4100
-Wire Wire Line
-	4800 4750 4800 5200
-Wire Wire Line
-	4800 5200 4250 5200
-Wire Wire Line
-	4450 4700 4450 4900
-Wire Wire Line
-	7300 4250 7300 4100
-Wire Wire Line
-	7300 4750 7100 4750
-Wire Wire Line
-	7100 4750 7100 4400
-Wire Wire Line
-	7100 4400 6850 4400
-Wire Wire Line
-	4450 4900 7600 4900
-Wire Wire Line
-	7600 4900 7600 4500
-Connection ~ 6850 4900
-Wire Wire Line
-	6600 4400 6600 5000
-Wire Wire Line
-	7100 5000 7100 4900
-Connection ~ 7100 4900
 $Comp
 L GND #PWR111
@@
 Text HLabel 4250 5200 0    60   Input ~ 0
 PA5
-NoConn ~ 5350 4400
 $Comp
 L R R69
