File: design/Power Supplies.sch (KiCad schematic (older format))
At the start: 11 parts, among them U10 LM2941S, U9 TLE4275

Commit message: revise schema according to Jaguar & Ravage project, eliminate as many errors as possible which were inherited from Puma board. Remove VSS interface, narrow band O2 interface, AC relay output, AC signal input. Make fuel injection configurable which can be batch fired or semi sequential fired
Parts:
- removed C43: 22uF, symbol C
- removed R69: 33K, symbol R
- removed R70: 29K4, symbol R
- removed R71: 10K, symbol R
- removed U10: LM2941S, symbol LM2941S
- added C43: 10uF, C1V7, symbol CAPAPOL
- added C52: 22uF, symbol C
- added C53: .1uF, C1V7, symbol C
- added D? (x2): ZENER, symbol ZENER
- added U10: TLE4275, symbol TLE4275
- C44: value 470nF -> .1uF; footprint (none) -> C1V7; Field1 (none) -> newark,56K3664; Field2 (none) -> vendor1, smd w hem; Field3 (none) -> vendor2, thru w hem; Field4 (none) -> vendor2, smd w hem; Field5 (none) -> 50,V; Field6 (none) -> 20,%; Field7 (none) -> multilayer ceramic; Field8 (none) -> other,more,stuff
Connections:
- net labels removed: PA5
- wire segments 27 -> 11
Other:
- note added: "Switched power regulator"
- note removed: "Switched power regulator with shutdown pin"
