File: design/U_Connector.sch (KiCad schematic (older format))
At the start: 3 parts

Commit message: prepare branch doing the I/O board prototyping
Connections:
- net labels added: +12V_SWITCHED
Changed lines of the file:
@@
-EESchema Schematic File Version 2  date 13/10/2011 15:17:47
+EESchema Schematic File Version 2  date 19/10/2011 09:07:12
 LIBS:power
 LIBS:device
@@
 Sheet 2 12
 Title ""
-Date "13 oct 2011"
+Date "19 oct 2011"
 Rev "0.01"
 Comp ""
@@
 Comment4 ""
 $EndDescr
+$Comp
+L +12V_SWITCHED #PWR?
+U 1 1 4E9E22BA
+P 3550 4950
+F 0 "#PWR?" H 3550 4900 20  0001 C CNN
+F 1 "+12V_SWITCHED" H 3550 5050 30  0000 C CNN
+	1    3550 4950
+	1    0    0    -1
+$EndComp
+$Comp
+L +12V_SWITCHED #PWR?
+U 1 1 4E9E2255
+P 3550 6250
+F 0 "#PWR?" H 3550 6200 20  0001 C CNN
+F 1 "+12V_SWITCHED" H 3550 6350 30  0000 C CNN
+	1    3550 6250
+	1    0    0    -1
+$EndComp
 NoConn ~ 3000 2800
 Text Notes 3900 2250 0    60   ~ 0
@@
 	1    0    0    -1
 $EndComp
-$Comp
-L +5V_SWITCHED #PWR?
-U 1 1 4E95B36C
-P 3550 6250
-F 0 "#PWR?" H 3550 6200 20  0001 C CNN
-F 1 "+5V_SWITCHED" H 3550 6350 30  0000 C CNN
-	1    3550 6250
-	1    0    0    -1
-$EndComp
 NoConn ~ 9100 2200
 $Comp
@@
 	1    0    0    -1
 $EndComp
-$Comp
-L +5V_SWITCHED #PWR?
-U 1 1 4E95B1B3
-P 3550 4950
-F 0 "#PWR?" H 3550 4900 20  0001 C CNN
-F 1 "+5V_SWITCHED" H 3550 5050 30  0000 C CNN
-	1    3550 4950
-	1    0    0    -1
-$EndComp

Commit message: decide to put CPU on mainboard, drop core board design
Parts:
- removed P?: CONN_2, symbol CONN_2
- removed P?: CONN_4, symbol CONN_4
Connections:
- net labels removed: RFU_Injector_#1, RFU_Injector_#2, RFU_Injector_#3, RPM1+, RPM1-
- no-connect marks 9 -> 8
Other:
- note added: "all ground should be meet together"
- note removed: "RFU cam signal providing\nengine phase info"
- note removed: "RFU injector interface\nfor sequencial injection"
Changed lines of the file:
@@
-EESchema Schematic File Version 2  date 19/10/2011 09:07:12
+EESchema Schematic File Version 2  date 27/12/2011 00:52:12
 LIBS:power
 LIBS:device
@@
 LIBS:contrib
 LIBS:valves
-LIBS:freeEMS_lib
-LIBS:catsquirt_ioboard-cache
+LIBS:mainboard-cache
 EELAYER 25  0
 EELAYER END
 $Descr A4 11700 8267
-Sheet 2 12
-Title ""
-Date "19 oct 2011"
+Sheet 3 12
+Title "OEM harness interface"
+Date "26 dec 2011"
 Rev "0.01"
-Comp ""
+Comp "diyefi.org"
 Comment1 ""
 Comment2 ""
@@
 Comment4 ""
 $EndDescr
+Text Notes 1350 4350 0    60   ~ 0
+all ground should be meet together
 $Comp
 L +12V_SWITCHED #PWR?
@@
 F 1 "+12V_SWITCHED" H 3550 6350 30  0000 C CNN
 	1    3550 6250
-	1    0    0    -1
-$EndComp
-NoConn ~ 3000 2800
-Text Notes 3900 2250 0    60   ~ 0
-RFU cam signal providing\nengine phase info
-Text Notes 2300 2250 0    60   ~ 0
-RFU injector interface\nfor sequencial injection
-$Comp
-L CONN_4 P?
-U 1 1 4E95B4F9
-P 3350 2650
-F 0 "P?" V 3300 2650 50  0000 C CNN
-F 1 "CONN_4" V 3400 2650 50  0000 C CNN
-	1    3350 2650
-	1    0    0    -1
-$EndComp
-$Comp
-L CONN_2 P?
-U 1 1 4E95B4EB
-P 4750 2600
-F 0 "P?" V 4700 2600 40  0000 C CNN
-F 1 "CONN_2" V 4800 2600 40  0000 C CNN
-	1    4750 2600
 	1    0    0    -1
 $EndComp
@@
 Text HLabel 4500 3800 0    60   Input ~ 0
 GAS_VENTI_VALVE
-Text HLabel 4400 2700 0    60   Input ~ 0
-RPM1-
-Text HLabel 4400 2500 0    60   Input ~ 0
-RPM1+
 Text HLabel 4450 4300 0    60   Input ~ 0
 RPM0-
@@
 Text HLabel 4450 5700 0    60   Input ~ 0
 IAT
-Text HLabel 3000 2700 0    60   Input ~ 0
-RFU_Injector_#3
-Text HLabel 3000 2600 0    60   Input ~ 0
-RFU_Injector_#2
-Text HLabel 3000 2500 0    60   Input ~ 0
-RFU_Injector_#1
 Text HLabel 4450 4900 0    60   Input ~ 0
 INJECTOR1-4

Commit message: revise schema to be full pin compatible with stock ECU
Parts:
- gave numbers to parts that had none: 1
Connections:
- net labels added: ADCGND, IGNGND, LSGND
- net labels removed: HCURGND, SENSORGND
- wire segments 67 -> 64
- no-connect marks 8 -> 9
Other:
- note removed: "all ground should be meet together"
Changed lines of the file:
@@
-EESchema Schematic File Version 2  date 27/12/2011 00:52:12
+EESchema Schematic File Version 2  date 02/01/2012 14:25:41
 LIBS:power
 LIBS:device
@@
 EELAYER END
 $Descr A4 11700 8267
-Sheet 3 12
+Sheet 4 12
 Title "OEM harness interface"
-Date "26 dec 2011"
+Date "2 jan 2012"
 Rev "0.01"
 Comp "diyefi.org"
@@
 Comment4 ""
 $EndDescr
-Text Notes 1350 4350 0    60   ~ 0
-all ground should be meet together
-$Comp
-L +12V_SWITCHED #PWR?
-U 1 1 4E9E22BA
-P 3550 4950
-F 0 "#PWR?" H 3550 4900 20  0001 C CNN
-F 1 "+12V_SWITCHED" H 3550 5050 30  0000 C CNN
-	1    3550 4950
-	1    0    0    -1
-$EndComp
-$Comp
-L +12V_SWITCHED #PWR?
+$Comp
+L GND #PWR?
+U 1 1 4F014DC6
+P 3550 5200
+F 0 "#PWR?" H 3550 5200 30  0001 C CNN
+F 1 "GND" H 3550 5130 30  0001 C CNN
+	1    3550 5200
+	1    0    0    -1
+$EndComp
+$Comp
+L LSGND #PWR?
+U 1 1 4F014D72
+P 3550 4650
+F 0 "#PWR?" H 3550 4650 40  0001 C CNN
+F 1 "LSGND" H 3550 4580 40  0000 C CNN
+	1    3550 4650
+	1    0    0    -1
+$EndComp
+NoConn ~ 7400 2200
+$Comp
+L ADCGND #PWR037
+U 1 1 4EFDEA8C
+P 3550 5650
+F 0 "#PWR037" H 3550 5650 40  0001 C CNN
+F 1 "ADCGND" H 3550 5580 40  0000 C CNN
+	1    3550 5650
+	1    0    0    -1
+$EndComp
+Wire Wire Line
+	3550 4250 3550 4200
+$Comp
+L ADCGND #PWR039
+U 1 1 4EFDE89C
+P 3550 4250
+F 0 "#PWR039" H 3550 4250 40  0001 C CNN
+F 1 "ADCGND" H 3550 4180 40  0000 C CNN
+	1    3550 4250
+	1    0    0    -1
+$EndComp
+$Comp
+L IGNGND #PWR040
+U 1 1 4EFDE808
+P 3550 3700
+F 0 "#PWR040" H 3550 3700 40  0001 C CNN
+F 1 "IGNGND" H 3550 3630 40  0000 C CNN
+	1    3550 3700
+	1    0    0    -1
+$EndComp
+$Comp
+L +12V_SWITCHED #PWR041
 U 1 1 4E9E2255
 P 3550 6250
-F 0 "#PWR?" H 3550 6200 20  0001 C CNN
+F 0 "#PWR041" H 3550 6200 20  0001 C CNN
 F 1 "+12V_SWITCHED" H 3550 6350 30  0000 C CNN
 	1    3550 6250
@@
 	7600 5200 4450 5200
 Wire Wire Line
-	7400 2200 7400 5000
-Wire Wire Line
-	7400 5000 3550 5000
-Wire Wire Line
-	3550 5000 3550 4950
-Wire Wire Line
 	5800 2200 5800 3600
 Wire Wire Line
@@
 	7200 4800 7200 2200
 Wire Wire Line
-	6600 4200 3550 4200
+	3550 4200 6600 4200
 Wire Wire Line
 	6600 4200 6600 2200
 Wire Wire Line
-	3550 4200 3550 4250
-Wire Wire Line
 	3550 4650 3550 4600
 Wire Wire Line
@@
 Wire Wire Line
 	9300 6300 9300 2200
-$Comp
-L HCURGND #PWR?
-U 1 1 4E95B431
-P 3550 3700
-F 0 "#PWR?" H 3550 3700 40  0001 C CNN
-F 1 "HCURGND" H 3550 3630 40  0000 C CNN
-	1    3550 3700
-	1    0    0    -1
-$EndComp
 NoConn ~ 9100 2200
 $Comp
-L SENSORGND #PWR?
-U 1 1 4E95B2AF
-P 3550 5650
-F 0 "#PWR?" H 3550 5650 40  0001 C CNN
-F 1 "SENSORGND" H 3550 5580 40  0000 C CNN
-	1    3550 5650
-	1    0    0    -1
-$EndComp
-$Comp
-L SENSORGND #PWR?
-U 1 1 4E95B1D6
-P 3550 5200
-F 0 "#PWR?" H 3550 5200 40  0001 C CNN
-F 1 "SENSORGND" H 3550 5130 40  0000 C CNN
-	1    3550 5200
-	1    0    0    -1
-$EndComp
-$Comp
-L GND #PWR?
-U 1 1 4E95B11C
-P 3550 4650
-F 0 "#PWR?" H 3550 4650 30  0001 C CNN
-F 1 "GND" H 3550 4580 30  0001 C CNN
-	1    3550 4650
-	1    0    0    -1
-$EndComp
-$Comp
-L SENSORGND #PWR?
-U 1 1 4E95B0BF
-P 3550 4250
-F 0 "#PWR?" H 3550 4250 40  0001 C CNN
-F 1 "SENSORGND" H 3550 4180 40  0000 C CNN
-	1    3550 4250
-	1    0    0    -1
-$EndComp
-$Comp
-L +5V_SWITCHED #PWR?
+L +5V_SWITCHED #PWR042
 U 1 1 4E95B079
 P 3550 4550
-F 0 "#PWR?" H 3550 4500 20  0001 C CNN
+F 0 "#PWR042" H 3550 4500 20  0001 C CNN
 F 1 "+5V_SWITCHED" H 3550 4650 30  0000 C CNN
 	1    3550 4550
@@
 NoConn ~ 6000 2200
 $Comp
-L BOSCH_MP5.2_37PIN P?
+L BOSCH_MP5.2_37PIN P3
 U 1 1 4E95964B
 P 6650 1850
-F 0 "P?" V 6800 1200 60  0000 C CNN
+F 0 "P3" V 6800 1200 60  0000 C CNN
 F 1 "BOSCH_MP5.2_37PIN" V 6700 1150 60  0000 C CNN
 	1    6650 1850

Commit message: use max9924 to replace ncv1124, add narrow band oxygen sensor differential input circuit, put all component into PCB edge
Connections:
- net labels added: NBO2+, NBO2-
- net labels removed: EGO
- wire segments 64 -> 62
Changed lines of the file:
@@
-EESchema Schematic File Version 2  date 14/01/2012 13:46:11
+EESchema Schematic File Version 2  date 21/01/2012 01:12:26
 LIBS:power
 LIBS:device
@@
 LIBS:contrib
 LIBS:valves
+LIBS:freeEMS_lib
 LIBS:mainboard-cache
 EELAYER 25  0
 EELAYER END
 $Descr A4 11700 8267
-Sheet 4 12
+Sheet 6 12
 Title "OEM harness interface"
-Date "14 jan 2012"
+Date "20 jan 2012"
 Rev "0.01"
 Comp "diyefi.org"
@@
 Comment4 ""
 $EndDescr
-$Comp
-L GND #PWR40
+Wire Wire Line
+	3550 4350 3550 4400
+Wire Wire Line
+	3550 4400 6800 4400
+Wire Wire Line
+	3550 3650 3550 3600
+Wire Wire Line
+	8900 2200 8900 6200
+Wire Wire Line
+	8900 6200 4450 6200
+Wire Wire Line
+	8600 2200 8600 6000
+Wire Wire Line
+	8600 6000 4450 6000
+Wire Wire Line
+	8400 2200 8400 5800
+Wire Wire Line
+	8400 5800 4450 5800
+Wire Wire Line
+	8200 2200 8200 5600
+Wire Wire Line
+	8200 5600 3550 5600
+Wire Wire Line
+	3550 5600 3550 5700
+Wire Wire Line
+	7900 2200 7900 5400
+Wire Wire Line
+	7900 5400 4450 5400
+Wire Wire Line
+	7600 2200 7600 5200
+Wire Wire Line
+	7600 5200 4450 5200
+Wire Wire Line
+	5800 2200 5800 3600
+Wire Wire Line
+	5800 3600 3550 3600
+Wire Wire Line
+	7000 2200 7000 4600
+Wire Wire Line
+	6800 4400 6800 2200
+Wire Wire Line
+	7300 2200 7300 4900
+Wire Wire Line
+	7300 4900 4450 4900
+Wire Wire Line
+	7100 2200 7100 4700
+Wire Wire Line
+	7100 4700 4450 4700
+Wire Wire Line
+	6700 2200 6700 4300
+Wire Wire Line
+	6700 4300 4450 4300
+Wire Wire Line
+	6300 2200 6300 4000
+Wire Wire Line
+	6300 4000 4500 4000
+Wire Wire Line
+	6100 2200 6100 3800
+Wire Wire Line
+	6100 3800 4500 3800
+Wire Wire Line
+	4500 3700 5900 3700
+Wire Wire Line
+	5900 3700 5900 2200
+Wire Wire Line
+	4500 3900 6200 3900
+Wire Wire Line
+	6200 3900 6200 2200
+Wire Wire Line
+	4500 4100 6500 4100
+Wire Wire Line
+	6500 4100 6500 2200
+Wire Wire Line
+	4450 4500 6900 4500
+Wire Wire Line
+	6900 4500 6900 2200
+Wire Wire Line
+	4450 4800 7200 4800
+Wire Wire Line
+	7200 4800 7200 2200
+Wire Wire Line
+	4500 4200 6600 4200
+Wire Wire Line
+	6600 4200 6600 2200
+Wire Wire Line
+	3550 4700 3550 4600
+Wire Wire Line
+	3550 4600 7000 4600
+Wire Wire Line
+	5700 2200 5700 3500
+Wire Wire Line
+	5700 3500 4500 3500
+Wire Wire Line
+	3550 5200 3550 5100
+Wire Wire Line
+	3550 5100 7500 5100
+Wire Wire Line
+	7500 5100 7500 2200
+Wire Wire Line
+	4450 5300 7800 5300
+Wire Wire Line
+	7800 5300 7800 2200
+Wire Wire Line
+	4450 5500 8100 5500
+Wire Wire Line
+	8100 5500 8100 2200
+Wire Wire Line
+	4450 5700 8300 5700
+Wire Wire Line
+	8300 5700 8300 2200
+Wire Wire Line
+	4450 5900 8500 5900
+Wire Wire Line
+	8500 5900 8500 2200
+Wire Wire Line
+	4450 6100 8800 6100
+Wire Wire Line
+	8800 6100 8800 2200
+Wire Wire Line
+	3550 6250 3550 6300
+Wire Wire Line
+	3550 6300 9300 6300
+Wire Wire Line
+	9300 6300 9300 2200
+Text HLabel 4500 4200 0    60   Input ~ 0
+NBO2-
+$Comp
+L GND #PWR69
 U 1 1 4F014DC6
 P 3550 5200
-F 0 "#PWR40" H 3550 5200 30  0001 C CNN
+F 0 "#PWR69" H 3550 5200 30  0001 C CNN
 F 1 "GND" H 3550 5130 30  0001 C CNN
 	1    3550 5200
@@
 $EndComp
 $Comp
-L LSGND #PWR39
+L LSGND #PWR68
 U 1 1 4F014D72
-P 3550 4650
-F 0 "#PWR39" H 3550 4650 40  0001 C CNN
-F 1 "LSGND" H 3550 4580 40  0000 C CNN
-	1    3550 4650
+P 3550 4700
+F 0 "#PWR68" H 3550 4700 40  0001 C CNN
+F 1 "LSGND" H 3550 4630 40  0000 C CNN
+	1    3550 4700
 	1    0    0    -1
 $EndComp
 NoConn ~ 7400 2200
 $Comp
-L ADCGND #PWR41
+L ADCGND #PWR70
 U 1 1 4EFDEA8C
-P 3550 5650
-F 0 "#PWR41" H 3550 5650 40  0001 C CNN
-F 1 "ADCGND" H 3550 5580 40  0000 C CNN
-	1    3550 5650
-	1    0    0    -1
-$EndComp
-Wire Wire Line
-	3550 4250 3550 4200
-$Comp
-L ADCGND #PWR37
-U 1 1 4EFDE89C
-P 3550 4250
-F 0 "#PWR37" H 3550 4250 40  0001 C CNN
-F 1 "ADCGND" H 3550 4180 40  0000 C CNN
-	1    3550 4250
-	1    0    0    -1
-$EndComp
-$Comp
-L IGNGND #PWR36
+P 3550 5700
+F 0 "#PWR70" H 3550 5700 40  0001 C CNN
+F 1 "ADCGND" H 3550 5630 40  0000 C CNN
+	1    3550 5700
+	1    0    0    -1
+$EndComp
+$Comp
+L IGNGND #PWR66
 U 1 1 4EFDE808
-P 3550 3700
-F 0 "#PWR36" H 3550 3700 40  0001 C CNN
-F 1 "IGNGND" H 3550 3630 40  0000 C CNN
-	1    3550 3700
-	1    0    0    -1
-$EndComp
-$Comp
-L +12V_SWITCHED #PWR42
+P 3550 3650
+F 0 "#PWR66" H 3550 3650 40  0001 C CNN
+F 1 "IGNGND" H 3550 3580 40  0000 C CNN
+	1    3550 3650
+	1    0    0    -1
+$EndComp
+$Comp
+L +12V_SWITCHED #PWR71
 U 1 1 4E9E2255
 P 3550 6250
-F 0 "#PWR42" H 3550 6200 20  0001 C CNN
+F 0 "#PWR71" H 3550 6200 20  0001 C CNN
 F 1 "+12V_SWITCHED" H 3550 6350 30  0000 C CNN
 	1    3550 6250
 	1    0    0    -1
 $EndComp
-Wire Wire Line
-	3550 3700 3550 3600
-Wire Wire Line
-	8900 2200 8900 6200
-Wire Wire Line
-	8900 6200 4450 6200
-Wire Wire Line
-	8600 2200 8600 6000
-Wire Wire Line
-	8600 6000 4450 6000
-Wire Wire Line
-	8400 2200 8400 5800
-Wire Wire Line
-	8400 5800 4450 5800
-Wire Wire Line
-	8200 2200 8200 5600
-Wire Wire Line
-	8200 5600 3550 5600
-Wire Wire Line
-	3550 5600 3550 5650
-Wire Wire Line
-	7900 2200 7900 5400
-Wire Wire Line
-	7900 5400 4450 5400
-Wire Wire Line
-	7600 2200 7600 5200
-Wire Wire Line
-	7600 5200 4450 5200
-Wire Wire Line
-	5800 2200 5800 3600
-Wire Wire Line
-	5800 3600 3550 3600
-Wire Wire Line
-	7000 2200 7000 4600
-Wire Wire Line
-	6800 2200 6800 4400
-Wire Wire Line
-	6800 4400 4000 4400
-Wire Wire Line
-	4000 4400 4000 4550
-Wire Wire Line
-	4000 4550 3550 4550
-Wire Wire Line
-	7300 2200 7300 4900
-Wire Wire Line
-	7300 4900 4450 4900
-Wire Wire Line
-	7100 2200 7100 4700
-Wire Wire Line
-	7100 4700 4450 4700
-Wire Wire Line
-	6700 2200 6700 4300
-Wire Wire Line
-	6700 4300 4450 4300
-Wire Wire Line
-	6300 2200 6300 4000
-Wire Wire Line
-	6300 4000 4500 4000
-Wire Wire Line
-	6100 2200 6100 3800
-Wire Wire Line
-	6100 3800 4500 3800
-Wire Wire Line
-	4500 3700 5900 3700
-Wire Wire Line
-	5900 3700 5900 2200
-Wire Wire Line
-	4500 3900 6200 3900
-Wire Wire Line
-	6200 3900 6200 2200
-Wire Wire Line
-	4500 4100 6500 4100
-Wire Wire Line
-	6500 4100 6500 2200
-Wire Wire Line
-	4450 4500 6900 4500
-Wire Wire Line
-	6900 4500 6900 2200
-Wire Wire Line
-	4450 4800 7200 4800
-Wire Wire Line
-	7200 4800 7200 2200
-Wire Wire Line
-	3550 4200 6600 4200
-Wire Wire Line
-	6600 4200 6600 2200
-Wire Wire Line
-	3550 4650 3550 4600
-Wire Wire Line
-	3550 4600 7000 4600
-Wire Wire Line
-	5700 2200 5700 3500
-Wire Wire Line
-	5700 3500 4500 3500
-Wire Wire Line
-	3550 5200 3550 5100
-Wire Wire Line
-	3550 5100 7500 5100
-Wire Wire Line
-	7500 5100 7500 2200
-Wire Wire Line
-	4450 5300 7800 5300
-Wire Wire Line
-	7800 5300 7800 2200
-Wire Wire Line
-	4450 5500 8100 5500
-Wire Wire Line
-	8100 5500 8100 2200
-Wire Wire Line
-	4450 5700 8300 5700
-Wire Wire Line
-	8300 5700 8300 2200
-Wire Wire Line
-	4450 5900 8500 5900
-Wire Wire Line
-	8500 5900 8500 2200
-Wire Wire Line
-	4450 6100 8800 6100
-Wire Wire Line
-	8800 6100 8800 2200
-Wire Wire Line
-	3550 6250 3550 6300
-Wire Wire Line
-	3550 6300 9300 6300
-Wire Wire Line
-	9300 6300 9300 2200
 NoConn ~ 9100 2200
 $Comp
-L +5V_SWITCHED #PWR38
+L +5V_SWITCHED #PWR67
 U 1 1 4E95B079
-P 3550 4550
-F 0 "#PWR38" H 3550 4500 20  0001 C CNN
-F 1 "+5V_SWITCHED" H 3550 4650 30  0000 C CNN
-	1    3550 4550
+P 3550 4350
+F 0 "#PWR67" H 3550 4300 20  0001 C CNN
+F 1 "+5V_SWITCHED" H 3550 4450 30  0000 C CNN
+	1    3550 4350
 	1    0    0    -1
 $EndComp
@@
 MAP
 Text HLabel 4450 5800 0    60   Input ~ 0
-EGO
+NBO2+
 Text HLabel 4450 5900 0    60   Input ~ 0
 TPS

Commit message: make new footprint for max9924 & lm9040, add can bus interface, generate new netlist
Changed lines of the file:
@@
-EESchema Schematic File Version 2  date 21/01/2012 01:12:26
+EESchema Schematic File Version 2  date 24/01/2012 16:34:51
 LIBS:power
 LIBS:device
@@
 Sheet 6 12
 Title "OEM harness interface"
-Date "20 jan 2012"
+Date "24 jan 2012"
 Rev "0.01"
 Comp "diyefi.org"
@@
 	3550 4400 6800 4400
 Wire Wire Line
-	3550 3650 3550 3600
+	3550 3700 3550 3600
 Wire Wire Line
 	8900 2200 8900 6200
@@
 NBO2-
 $Comp
-L GND #PWR69
+L GND #PWR067
 U 1 1 4F014DC6
 P 3550 5200
-F 0 "#PWR69" H 3550 5200 30  0001 C CNN
+F 0 "#PWR067" H 3550 5200 30  0001 C CNN
 F 1 "GND" H 3550 5130 30  0001 C CNN
 	1    3550 5200
@@
 $EndComp
 $Comp
-L LSGND #PWR68
+L LSGND #PWR068
 U 1 1 4F014D72
 P 3550 4700
-F 0 "#PWR68" H 3550 4700 40  0001 C CNN
+F 0 "#PWR068" H 3550 4700 40  0001 C CNN
 F 1 "LSGND" H 3550 4630 40  0000 C CNN
 	1    3550 4700
@@
 NoConn ~ 7400 2200
 $Comp
-L ADCGND #PWR70
+L ADCGND #PWR069
 U 1 1 4EFDEA8C
 P 3550 5700
-F 0 "#PWR70" H 3550 5700 40  0001 C CNN
+F 0 "#PWR069" H 3550 5700 40  0001 C CNN
 F 1 "ADCGND" H 3550 5630 40  0000 C CNN
 	1    3550 5700
@@
 $EndComp
 $Comp
-L IGNGND #PWR66
+L IGNGND #PWR070
 U 1 1 4EFDE808
-P 3550 3650
-F 0 "#PWR66" H 3550 3650 40  0001 C CNN
-F 1 "IGNGND" H 3550 3580 40  0000 C CNN
-	1    3550 3650
-	1    0    0    -1
-$EndComp
-$Comp
-L +12V_SWITCHED #PWR71
+P 3550 3700
+F 0 "#PWR070" H 3550 3700 40  0001 C CNN
+F 1 "IGNGND" H 3550 3630 40  0000 C CNN
+	1    3550 3700
+	1    0    0    -1
+$EndComp
+$Comp
+L +12V_SWITCHED #PWR071
 U 1 1 4E9E2255
 P 3550 6250
-F 0 "#PWR71" H 3550 6200 20  0001 C CNN
+F 0 "#PWR071" H 3550 6200 20  0001 C CNN
 F 1 "+12V_SWITCHED" H 3550 6350 30  0000 C CNN
 	1    3550 6250
@@
 NoConn ~ 9100 2200
 $Comp
-L +5V_SWITCHED #PWR67
+L +5V_SWITCHED #PWR072
 U 1 1 4E95B079
 P 3550 4350
-F 0 "#PWR67" H 3550 4300 20  0001 C CNN
+F 0 "#PWR072" H 3550 4300 20  0001 C CNN
 F 1 "+5V_SWITCHED" H 3550 4450 30  0000 C CNN
 	1    3550 4350
