File: design/U_Connector.sch (KiCad schematic (older format))
At the start: 1 part, among them P3 BOSCH_MP5.2_37PIN

Commit message: revise schema according to Jaguar & Ravage project, eliminate as many errors as possible which were inherited from Puma board. Remove VSS interface, narrow band O2 interface, AC relay output, AC signal input. Make fuel injection configurable which can be batch fired or semi sequential fired
Parts:
- added P5: AC open, symbol CONN_2
Connections:
- net labels removed: AC_CLUTCH_RELAY, AC_SIGNAL, CHECK_ENGINE, K_WIRE, L_WIRE, MAP, NBO2+, NBO2-, SPEED_SENSOR
- wire segments 62 -> 48
- no-connect marks 9 -> 17
Other:
- note added: "my ECU is not responsible to control AC\njust solder pin 23 to low side ground"
Changed lines of the file:
@@
-EESchema Schematic File Version 2  date 29/01/2012 19:39:37
+EESchema Schematic File Version 2  date 02/02/2012 00:51:37
 LIBS:power
 LIBS:device
@@
 EELAYER END
 $Descr A4 11700 8267
-Sheet 6 12
+Sheet 3 10
 Title "OEM harness interface"
-Date "24 jan 2012"
+Date "1 feb 2012"
 Rev "0.01"
 Comp "diyefi.org"
@@
 Comment4 ""
 $EndDescr
-Wire Wire Line
-	3550 4350 3550 4400
-Wire Wire Line
-	3550 4400 6800 4400
-Wire Wire Line
-	3550 3700 3550 3600
-Wire Wire Line
-	8900 2200 8900 6200
-Wire Wire Line
-	8900 6200 4450 6200
-Wire Wire Line
-	8600 2200 8600 6000
-Wire Wire Line
-	8600 6000 4450 6000
-Wire Wire Line
-	8400 2200 8400 5800
-Wire Wire Line
-	8400 5800 4450 5800
-Wire Wire Line
-	8200 2200 8200 5600
-Wire Wire Line
-	8200 5600 3550 5600
-Wire Wire Line
-	3550 5600 3550 5700
-Wire Wire Line
-	7900 2200 7900 5400
-Wire Wire Line
-	7900 5400 4450 5400
-Wire Wire Line
-	7600 2200 7600 5200
-Wire Wire Line
-	7600 5200 4450 5200
-Wire Wire Line
-	5800 2200 5800 3600
+Text Notes 4750 1500 0    30   ~ 0
+my ECU is not responsible to control AC\njust solder pin 23 to low side ground
+Wire Wire Line
+	7900 2200 7900 2600
+Wire Wire Line
+	7900 2600 5300 2600
+Wire Wire Line
+	5300 2600 5300 2100
+Wire Wire Line
+	9300 2200 9300 6300
+Wire Wire Line
+	9300 6300 3550 6300
+Wire Wire Line
+	3550 6300 3550 6250
+Wire Wire Line
+	8500 2200 8500 5900
+Wire Wire Line
+	8500 5900 4450 5900
+Wire Wire Line
+	8300 2200 8300 5700
+Wire Wire Line
+	8300 5700 4450 5700
+Wire Wire Line
+	8100 2200 8100 5500
+Wire Wire Line
+	8100 5500 4450 5500
+Wire Wire Line
+	7500 2200 7500 5100
+Wire Wire Line
+	7500 5100 3550 5100
+Wire Wire Line
+	3550 5100 3550 5200
+Wire Wire Line
+	4500 3500 5700 3500
+Wire Wire Line
+	5700 3500 5700 2200
+Wire Wire Line
+	3550 4600 7000 4600
+Wire Wire Line
+	3550 4600 3550 4700
+Wire Wire Line
+	6200 2200 6200 3900
+Wire Wire Line
+	6200 3900 4500 3900
+Wire Wire Line
+	5900 2200 5900 3700
+Wire Wire Line
+	5900 3700 4500 3700
+Wire Wire Line
+	4500 3800 6100 3800
+Wire Wire Line
+	6100 3800 6100 2200
+Wire Wire Line
+	4450 4300 6700 4300
+Wire Wire Line
+	6700 4300 6700 2200
+Wire Wire Line
+	4450 4700 7100 4700
+Wire Wire Line
+	7100 4700 7100 2200
+Wire Wire Line
+	4450 4900 7300 4900
+Wire Wire Line
+	7300 4900 7300 2200
+Wire Wire Line
+	6800 2200 6800 4400
+Wire Wire Line
+	7000 4600 7000 2200
 Wire Wire Line
 	5800 3600 3550 3600
 Wire Wire Line
-	7000 2200 7000 4600
-Wire Wire Line
-	6800 4400 6800 2200
-Wire Wire Line
-	7300 2200 7300 4900
-Wire Wire Line
-	7300 4900 4450 4900
-Wire Wire Line
-	7100 2200 7100 4700
-Wire Wire Line
-	7100 4700 4450 4700
-Wire Wire Line
-	6700 2200 6700 4300
-Wire Wire Line
-	6700 4300 4450 4300
-Wire Wire Line
-	6300 2200 6300 4000
-Wire Wire Line
-	6300 4000 4500 4000
-Wire Wire Line
-	6100 2200 6100 3800
-Wire Wire Line
-	6100 3800 4500 3800
-Wire Wire Line
-	4500 3700 5900 3700
-Wire Wire Line
-	5900 3700 5900 2200
-Wire Wire Line
-	4500 3900 6200 3900
-Wire Wire Line
-	6200 3900 6200 2200
-Wire Wire Line
-	4500 4100 6500 4100
-Wire Wire Line
-	6500 4100 6500 2200
-Wire Wire Line
-	4450 4500 6900 4500
-Wire Wire Line
-	6900 4500 6900 2200
-Wire Wire Line
-	4450 4800 7200 4800
-Wire Wire Line
-	7200 4800 7200 2200
-Wire Wire Line
-	4500 4200 6600 4200
-Wire Wire Line
-	6600 4200 6600 2200
-Wire Wire Line
-	3550 4700 3550 4600
-Wire Wire Line
-	3550 4600 7000 4600
-Wire Wire Line
-	5700 2200 5700 3500
-Wire Wire Line
-	5700 3500 4500 3500
-Wire Wire Line
-	3550 5200 3550 5100
-Wire Wire Line
-	3550 5100 7500 5100
-Wire Wire Line
-	7500 5100 7500 2200
-Wire Wire Line
-	4450 5300 7800 5300
-Wire Wire Line
-	7800 5300 7800 2200
-Wire Wire Line
-	4450 5500 8100 5500
-Wire Wire Line
-	8100 5500 8100 2200
-Wire Wire Line
-	4450 5700 8300 5700
-Wire Wire Line
-	8300 5700 8300 2200
-Wire Wire Line
-	4450 5900 8500 5900
-Wire Wire Line
-	8500 5900 8500 2200
-Wire Wire Line
-	4450 6100 8800 6100
-Wire Wire Line
-	8800 6100 8800 2200
-Wire Wire Line
-	3550 6250 3550 6300
-Wire Wire Line
-	3550 6300 9300 6300
-Wire Wire Line
-	9300 6300 9300 2200
-Text HLabel 4500 4200 0    60   Input ~ 0
-NBO2-
-$Comp
-L GND #PWR067
+	5800 3600 5800 2200
+Wire Wire Line
+	4450 5200 7600 5200
+Wire Wire Line
+	7600 5200 7600 2200
+Wire Wire Line
+	3550 5700 3550 5600
+Wire Wire Line
+	3550 5600 8200 5600
+Wire Wire Line
+	8200 5600 8200 2200
+Wire Wire Line
+	4450 6000 8600 6000
+Wire Wire Line
+	8600 6000 8600 2200
+Wire Wire Line
+	4450 6200 8900 6200
+Wire Wire Line
+	8900 6200 8900 2200
+Wire Wire Line
+	3550 3600 3550 3700
+Wire Wire Line
+	6800 4400 3550 4400
+Wire Wire Line
+	3550 4400 3550 4350
+Wire Wire Line
+	5100 2100 5100 2350
+$Comp
+L LSGND #PWR030
+U 1 1 4F290E5D
+P 5100 2350
+F 0 "#PWR030" H 5100 2350 40  0001 C CNN
+F 1 "LSGND" H 5100 2280 40  0000 C CNN
+	1    5100 2350
+	1    0    0    -1
+$EndComp
+$Comp
+L CONN_2 P5
+U 1 1 4F290E03
+P 5200 1750
+F 0 "P5" V 5150 1750 40  0000 C CNN
+F 1 "AC open" V 5250 1750 40  0000 C CNN
+	1    5200 1750
+	0    -1   -1   0
+$EndComp
+NoConn ~ 6500 2200
+NoConn ~ 8800 2200
+NoConn ~ 7200 2200
+NoConn ~ 6900 2200
+NoConn ~ 6300 2200
+NoConn ~ 8400 2200
+NoConn ~ 6600 2200
+NoConn ~ 7800 2200
+$Comp
+L GND #PWR031
 U 1 1 4F014DC6
 P 3550 5200
-F 0 "#PWR067" H 3550 5200 30  0001 C CNN
+F 0 "#PWR031" H 3550 5200 30  0001 C CNN
 F 1 "GND" H 3550 5130 30  0001 C CNN
 	1    3550 5200
@@
 $EndComp
 $Comp
-L LSGND #PWR068
+L LSGND #PWR032
 U 1 1 4F014D72
 P 3550 4700
-F 0 "#PWR068" H 3550 4700 40  0001 C CNN
+F 0 "#PWR032" H 3550 4700 40  0001 C CNN
 F 1 "LSGND" H 3550 4630 40  0000 C CNN
 	1    3550 4700
@@
 NoConn ~ 7400 2200
 $Comp
-L ADCGND #PWR069
+L ADCGND #PWR033
 U 1 1 4EFDEA8C
 P 3550 5700
-F 0 "#PWR069" H 3550 5700 40  0001 C CNN
+F 0 "#PWR033" H 3550 5700 40  0001 C CNN
 F 1 "ADCGND" H 3550 5630 40  0000 C CNN
 	1    3550 5700
@@
 $EndComp
 $Comp
-L IGNGND #PWR070
+L IGNGND #PWR034
 U 1 1 4EFDE808
 P 3550 3700
-F 0 "#PWR070" H 3550 3700 40  0001 C CNN
+F 0 "#PWR034" H 3550 3700 40  0001 C CNN
 F 1 "IGNGND" H 3550 3630 40  0000 C CNN
 	1    3550 3700
@@
 $EndComp
 $Comp
-L +12V_SWITCHED #PWR071
+L +12V_SWITCHED #PWR035
 U 1 1 4E9E2255
 P 3550 6250
-F 0 "#PWR071" H 3550 6200 20  0001 C CNN
+F 0 "#PWR035" H 3550 6200 20  0001 C CNN
 F 1 "+12V_SWITCHED" H 3550 6350 30  0000 C CNN
 	1    3550 6250
@@
 NoConn ~ 9100 2200
 $Comp
-L +5V_SWITCHED #PWR072
+L +5V_SWITCHED #PWR036
 U 1 1 4E95B079
 P 3550 4350
-F 0 "#PWR072" H 3550 4300 20  0001 C CNN
+F 0 "#PWR036" H 3550 4300 20  0001 C CNN
 F 1 "+5V_SWITCHED" H 3550 4450 30  0000 C CNN
 	1    3550 4350
@@
 	0    -1   -1   0
 $EndComp
-Text Notes 7650 1400 2    30   ~ 0
+Text Notes 7650 1400 2    60   ~ 0
 OEM ECU connector ripped\nfrom Bosch MP5.2
-Text HLabel 4450 4500 0    60   Input ~ 0
-L_WIRE
-Text HLabel 4450 4800 0    60   Input ~ 0
-K_WIRE
 Text HLabel 4500 3700 0    60   Input ~ 0
 FUEL_PUMP_RELAY
@@
 Text HLabel 4450 4700 0    60   Input ~ 0
 STEPPER_OPEN
-Text HLabel 4450 5400 0    60   Input ~ 0
-AC_CLUTCH_RELAY
 Text HLabel 4500 3800 0    60   Input ~ 0
 GAS_VENTI_VALVE
@@
 Text HLabel 4450 6000 0    60   Input ~ 0
 RPM0+
-Text HLabel 4450 5300 0    60   Input ~ 0
-CHECK_ENGINE
 Text HLabel 4500 3900 0    60   Input ~ 0
 TACH_OUT
-Text HLabel 4500 4100 0    60   Input ~ 0
-SPEED_SENSOR
-Text HLabel 4450 6100 0    60   Input ~ 0
-AC_SIGNAL
-Text HLabel 4500 4000 0    60   Input ~ 0
-MAP
-Text HLabel 4450 5800 0    60   Input ~ 0
-NBO2+
 Text HLabel 4450 5900 0    60   Input ~ 0
 TPS

Commit message: make new footprint for screw connector, redesign ignition gnd & all lowside gnd
Parts:
- added P4, P7: Gnd Option, symbol CONN_2
- renumbered P5 to P2
Connections:
- net labels added: AC clutch relay, EGO
- wire segments 48 -> 63
- no-connect marks 17 -> 16
Other:
- note added: "IGNGND and LSGND can be combined \nwith this screw connector. Build two\nidentical connector allow high current\nto be splitted to gnds. Prevent too much\n current flow through one pin"
- moved on the sheet: P2

Commit message: revise schema according to DeuceEFI's claim
Other:
- note added: "IGNGND and LSGND can be combined \nwith this screw connector. Build two\nidentical connector allow high current\nto be splitted to gnds. Prevent too much\n current flowing through one pin"
- note removed: "IGNGND and LSGND can be combined \nwith this screw connector. Build two\nidentical connector allow high current\nto be splitted to gnds. Prevent too much\n current flow through one pin"
Changed lines of the file:
@@
-EESchema Schematic File Version 2  date 07/02/2012 00:44:28
+EESchema Schematic File Version 2  date 08/02/2012 17:27:57
 LIBS:power
 LIBS:device
@@
 Sheet 2 10
 Title "OEM harness interface"
-Date "6 feb 2012"
+Date "8 feb 2012"
 Rev "0.01"
 Comp "diyefi.org"
@@
 $EndComp
 Text Notes 1950 1550 0    30   ~ 0
-IGNGND and LSGND can be combined \nwith this screw connector. Build two\nidentical connector allow high current\nto be splitted to gnds. Prevent too much\n current flow through one pin
+IGNGND and LSGND can be combined \nwith this screw connector. Build two\nidentical connector allow high current\nto be splitted to gnds. Prevent too much\n current flowing through one pin
 $Comp
 L LSGND #PWR05

Commit message: some layout work, very dirty
Parts:
- removed P7: Gnd Option, symbol CONN_2
Connections:
- wire segments 63 -> 57
Other:
- note added: "IGNGND and LSGND can be combined \nwith this screw connector, allow high \ncurrent to be splitted to gnds."
- note removed: "IGNGND and LSGND can be combined \nwith this screw connector. Build two\nidentical connector allow high current\nto be splitted to gnds. Prevent too much\n current flowing through one pin"
- moved on the sheet: P2, P4
Changed lines of the file:
@@
-EESchema Schematic File Version 2  date 08/02/2012 17:27:57
+EESchema Schematic File Version 2  date 06/03/2012 22:16:34
 LIBS:power
 LIBS:device
@@
 Sheet 2 10
 Title "OEM harness interface"
-Date "8 feb 2012"
+Date "11 feb 2012"
 Rev "0.01"
 Comp "diyefi.org"
@@
 NoConn ~ 6600 2200
 Wire Wire Line
-	4550 2500 4400 2500
-Wire Wire Line
-	4400 2500 4400 2250
+	3450 2650 3300 2650
+Wire Wire Line
+	3300 2650 3300 2400
 Wire Wire Line
 	4450 5350 7900 5350
@@
 	7900 5350 7900 2200
 Wire Wire Line
-	1750 2250 1750 2350
-Wire Wire Line
-	1750 2350 1500 2350
-Wire Wire Line
-	1500 2350 1500 2500
-Wire Wire Line
-	2150 2500 2150 2350
-Wire Wire Line
-	2150 2350 1950 2350
-Wire Wire Line
-	1950 2350 1950 2250
-Wire Wire Line
-	3000 2250 3000 2350
-Wire Wire Line
-	3000 2350 3200 2350
-Wire Wire Line
-	3200 2350 3200 2500
-Wire Wire Line
-	2550 2500 2550 2350
+	1900 2400 1900 2500
+Wire Wire Line
+	1900 2500 1650 2500
+Wire Wire Line
+	1650 2500 1650 2650
+Wire Wire Line
+	2350 2650 2350 2500
+Wire Wire Line
+	2350 2500 2100 2500
+Wire Wire Line
+	2100 2500 2100 2400
 Wire Wire Line
 	9300 2200 9300 6300
@@
 	3550 4400 3550 4350
 Wire Wire Line
-	4200 2250 4200 2500
+	3100 2400 3100 2650
 Wire Wire Line
 	8400 2200 8400 5800
 Wire Wire Line
 	8400 5800 4450 5800
-Wire Wire Line
-	2550 2350 2800 2350
-Wire Wire Line
-	2800 2350 2800 2250
-Text GLabel 4550 2500 2    60   Output ~ 0
+Text GLabel 3450 2650 2    60   Output ~ 0
 AC clutch relay
 Text GLabel 4450 5350 0    60   Output ~ 0
@@
 L PWR_FLAG #FLG01
 U 1 1 4F2FFC81
-P 2550 2350
-F 0 "#FLG01" H 2550 2620 30  0001 C CNN
-F 1 "PWR_FLAG" H 2550 2580 30  0000 C CNN
-	1    2550 2350
+P 1650 2500
+F 0 "#FLG01" H 1650 2770 30  0001 C CNN
+F 1 "PWR_FLAG" H 1650 2730 30  0000 C CNN
+	1    1650 2500
 	1    0    0    -1
 $EndComp
@@
 L PWR_FLAG #FLG02
 U 1 1 4F2FFC74
-P 2150 2350
-F 0 "#FLG02" H 2150 2620 30  0001 C CNN
-F 1 "PWR_FLAG" H 2150 2580 30  0000 C CNN
-	1    2150 2350
+P 2350 2500
+F 0 "#FLG02" H 2350 2770 30  0001 C CNN
+F 1 "PWR_FLAG" H 2350 2730 30  0000 C CNN
+	1    2350 2500
 	1    0    0    -1
 $EndComp
@@
 L IGNGND #PWR03
 U 1 1 4F2FF9A3
-P 1500 2500
-F 0 "#PWR03" H 1500 2500 40  0001 C CNN
-F 1 "IGNGND" H 1500 2430 40  0000 C CNN
-	1    1500 2500
+P 1650 2650
+F 0 "#PWR03" H 1650 2650 40  0001 C CNN
+F 1 "IGNGND" H 1650 2580 40  0000 C CNN
+	1    1650 2650
 	1    0    0    -1
 $EndComp
@@
 L LSGND #PWR04
 U 1 1 4F2FF9A2
-P 2150 2500
-F 0 "#PWR04" H 2150 2500 40  0001 C CNN
-F 1 "LSGND" H 2150 2430 40  0000 C CNN
-	1    2150 2500
+P 2350 2650
+F 0 "#PWR04" H 2350 2650 40  0001 C CNN
+F 1 "LSGND" H 2350 2580 40  0000 C CNN
+	1    2350 2650
 	1    0    0    -1
 $EndComp
@@
 L CONN_2 P4
 U 1 1 4F2FF9A1
-P 1850 1900
-F 0 "P4" V 1800 1900 40  0000 C CNN
-F 1 "Gnd Option" V 1900 1900 40  0000 C CNN
-	1    1850 1900
+P 2000 2050
+F 0 "P4" V 1950 2050 40  0000 C CNN
+F 1 "Gnd Option" V 2050 2050 40  0000 C CNN
+	1    2000 2050
 	0    -1   -1   0
 $EndComp
-$Comp
-L CONN_2 P7
-U 1 1 4F2FF830
-P 2900 1900
-F 0 "P7" V 2850 1900 40  0000 C CNN
-F 1 "Gnd Option" V 2950 1900 40  0000 C CNN
-	1    2900 1900
-	0    -1   -1   0
-$EndComp
-Text Notes 1950 1550 0    30   ~ 0
-IGNGND and LSGND can be combined \nwith this screw connector. Build two\nidentical connector allow high current\nto be splitted to gnds. Prevent too much\n current flowing through one pin
-$Comp
-L LSGND #PWR05
-U 1 1 4F2FF7D1
-P 3200 2500
-F 0 "#PWR05" H 3200 2500 40  0001 C CNN
-F 1 "LSGND" H 3200 2430 40  0000 C CNN
-	1    3200 2500
-	1    0    0    -1
-$EndComp
-$Comp
-L IGNGND #PWR06
-U 1 1 4F2FF7CD
-P 2550 2500
-F 0 "#PWR06" H 2550 2500 40  0001 C CNN
-F 1 "IGNGND" H 2550 2430 40  0000 C CNN
-	1    2550 2500
-	1    0    0    -1
-$EndComp
+Text Notes 1550 1800 0    30   ~ 0
+IGNGND and LSGND can be combined \nwith this screw connector, allow high \ncurrent to be splitted to gnds.
 Text HLabel 4450 5800 0    60   Output ~ 0
 EGO
-Text Notes 3850 1650 0    30   ~ 0
+Text Notes 2750 1800 0    30   ~ 0
 my ECU is not responsible to control AC\njust solder pin 23 to low side ground
 $Comp
-L LSGND #PWR07
+L LSGND #PWR05
 U 1 1 4F290E5D
-P 4200 2500
-F 0 "#PWR07" H 4200 2500 40  0001 C CNN
-F 1 "LSGND" H 4200 2430 40  0000 C CNN
-	1    4200 2500
+P 3100 2650
+F 0 "#PWR05" H 3100 2650 40  0001 C CNN
+F 1 "LSGND" H 3100 2580 40  0000 C CNN
+	1    3100 2650
 	1    0    0    -1
 $EndComp
@@
 L CONN_2 P2
 U 1 1 4F290E03
-P 4300 1900
-F 0 "P2" V 4250 1900 40  0000 C CNN
-F 1 "AC open" V 4350 1900 40  0000 C CNN
-	1    4300 1900
+P 3200 2050
+F 0 "P2" V 3150 2050 40  0000 C CNN
+F 1 "AC open" V 3250 2050 40  0000 C CNN
+	1    3200 2050
 	0    -1   -1   0
 $EndComp
@@
 NoConn ~ 7800 2200
 $Comp
-L GND #PWR08
+L GND #PWR06
 U 1 1 4F014DC6
 P 3550 5200
-F 0 "#PWR08" H 3550 5200 30  0001 C CNN
+F 0 "#PWR06" H 3550 5200 30  0001 C CNN
 F 1 "GND" H 3550 5130 30  0001 C CNN
 	1    3550 5200
@@
 $EndComp
 $Comp
-L LSGND #PWR09
+L LSGND #PWR07
 U 1 1 4F014D72
 P 3550 4700
-F 0 "#PWR09" H 3550 4700 40  0001 C CNN
+F 0 "#PWR07" H 3550 4700 40  0001 C CNN
 F 1 "LSGND" H 3550 4630 40  0000 C CNN
 	1    3550 4700
@@
 NoConn ~ 7400 2200
 $Comp
-L ADCGND #PWR010
+L ADCGND #PWR08
 U 1 1 4EFDEA8C
 P 3550 5700
-F 0 "#PWR010" H 3550 5700 40  0001 C CNN
+F 0 "#PWR08" H 3550 5700 40  0001 C CNN
 F 1 "ADCGND" H 3550 5630 40  0000 C CNN
 	1    3550 5700
@@
 $EndComp
 $Comp
-L IGNGND #PWR011
+L IGNGND #PWR09
 U 1 1 4EFDE808
 P 3550 3700
-F 0 "#PWR011" H 3550 3700 40  0001 C CNN
+F 0 "#PWR09" H 3550 3700 40  0001 C CNN
 F 1 "IGNGND" H 3550 3630 40  0000 C CNN
 	1    3550 3700
@@
 $EndComp
 $Comp
-L +12V_SWITCHED #PWR012
+L +12V_SWITCHED #PWR010
 U 1 1 4E9E2255
 P 3550 6250
-F 0 "#PWR012" H 3550 6200 20  0001 C CNN
+F 0 "#PWR010" H 3550 6200 20  0001 C CNN
 F 1 "+12V_SWITCHED" H 3550 6350 30  0000 C CNN
 	1    3550 6250
@@
 NoConn ~ 9100 2200
 $Comp
-L +5V_SWITCHED #PWR013
+L +5V_SWITCHED #PWR011
 U 1 1 4E95B079
 P 3550 4350
-F 0 "#PWR013" H 3550 4300 20  0001 C CNN
+F 0 "#PWR011" H 3550 4300 20  0001 C CNN
 F 1 "+5V_SWITCHED" H 3550 4450 30  0000 C CNN
 	1    3550 4350
