File: design/U_Igniter Outputs.sch (KiCad schematic (older format))
At the start: 21 parts

Commit message: revise schema to be full pin compatible with stock ECU
Parts:
- C30: renamed from C?; value C -> 0.1uF
- K2: renamed from K?; value CONN_3 -> jumper
- R34, R35: renamed from R?; value R -> 1K
- R36, R37: renamed from R?; value R -> 100K
- gave numbers to parts that had none: 15
Connections:
- net labels added: IGNGND
- net labels removed: HCURGND
Changed lines of the file:
@@
-EESchema Schematic File Version 2  date 27/12/2011 00:52:12
+EESchema Schematic File Version 2  date 02/01/2012 14:25:41
 LIBS:power
 LIBS:device
@@
 EELAYER END
 $Descr A4 11700 8267
-Sheet 5 12
-Title ""
-Date "26 dec 2011"
-Rev ""
-Comp ""
+Sheet 6 12
+Title "ignition module"
+Date "2 jan 2012"
+Rev "0.01"
+Comp "diyefi.org"
 Comment1 ""
 Comment2 ""
@@
 Comment4 ""
 $EndDescr
+Wire Wire Line
+	8900 5850 8900 4800
+$Comp
+L IGNGND #PWR059
+U 1 1 4EFDEBD7
+P 8900 5850
+F 0 "#PWR059" H 8900 5850 40  0001 C CNN
+F 1 "IGNGND" H 8900 5780 40  0000 C CNN
+	1    8900 5850
+	1    0    0    -1
+$EndComp
+$Comp
+L IGNGND #PWR060
+U 1 1 4EFDEBD2
+P 9000 3450
+F 0 "#PWR060" H 9000 3450 40  0001 C CNN
+F 1 "IGNGND" H 9000 3380 40  0000 C CNN
+	1    9000 3450
+	1    0    0    -1
+$EndComp
 Connection ~ 8000 1700
 Wire Wire Line
@@
 	6900 4400 6750 4400
 Wire Wire Line
-	8650 4800 8900 4800
+	8900 4800 8650 4800
 Wire Wire Line
 	8900 5000 8650 5000
@@
 Connection ~ 8650 5750
 Wire Wire Line
-	8900 4800 8900 5850
-Wire Wire Line
 	4900 3750 4900 3350
 Wire Wire Line
@@
 	7900 4350 7900 4100
 $Comp
-L R R?
+L R R38
 U 1 1 4E95AA74
 P 6850 4100
-F 0 "R?" V 6930 4100 50  0000 C CNN
+F 0 "R38" V 6930 4100 50  0000 C CNN
 F 1 "2K4" V 6850 4100 50  0000 C CNN
 	1    6850 4100
@@
 $EndComp
 $Comp
-L LED D?
+L LED D15
 U 1 1 4E95AA73
 P 7450 4100
-F 0 "D?" H 7450 4200 50  0000 C CNN
+F 0 "D15" H 7450 4200 50  0000 C CNN
 F 1 "LED" H 7450 4000 50  0000 C CNN
 	1    7450 4100
@@
 $EndComp
 $Comp
-L +12V_SWITCHED #PWR?
+L +12V_SWITCHED #PWR061
 U 1 1 4E95AA72
 P 6250 3900
-F 0 "#PWR?" H 6250 3850 20  0001 C CNN
+F 0 "#PWR061" H 6250 3850 20  0001 C CNN
 F 1 "+12V_SWITCHED" H 6250 4000 30  0000 C CNN
 	1    6250 3900
@@
 $EndComp
 $Comp
-L R R?
+L R R31
 U 1 1 4E95AA37
 P 6950 1700
-F 0 "R?" V 7030 1700 50  0000 C CNN
+F 0 "R31" V 7030 1700 50  0000 C CNN
 F 1 "2K4" V 6950 1700 50  0000 C CNN
 	1    6950 1700
@@
 $EndComp
 $Comp
-L LED D?
+L LED D14
 U 1 1 4E95AA36
 P 7550 1700
-F 0 "D?" H 7550 1800 50  0000 C CNN
+F 0 "D14" H 7550 1800 50  0000 C CNN
 F 1 "LED" H 7550 1600 50  0000 C CNN
 	1    7550 1700
@@
 $EndComp
 $Comp
-L +12V_SWITCHED #PWR?
+L +12V_SWITCHED #PWR062
 U 1 1 4E95AA35
 P 6350 1500
-F 0 "#PWR?" H 6350 1450 20  0001 C CNN
+F 0 "#PWR062" H 6350 1450 20  0001 C CNN
 F 1 "+12V_SWITCHED" H 6350 1600 30  0000 C CNN
 	1    6350 1500
@@
 $EndComp
 $Comp
-L +5V_SWITCHED #PWR?
+L +5V_SWITCHED #PWR063
 U 1 1 4E9456A3
 P 5900 4500
-F 0 "#PWR?" H 5900 4450 20  0001 C CNN
+F 0 "#PWR063" H 5900 4450 20  0001 C CNN
 F 1 "+5V_SWITCHED" H 5900 4600 30  0000 C CNN
 	1    5900 4500
@@
 $EndComp
 $Comp
-L +5V_SWITCHED #PWR?
+L +5V_SWITCHED #PWR064
 U 1 1 4E94565D
 P 5900 2250
-F 0 "#PWR?" H 5900 2200 20  0001 C CNN
+F 0 "#PWR064" H 5900 2200 20  0001 C CNN
 F 1 "+5V_SWITCHED" H 5900 2350 30  0000 C CNN
 	1    5900 2250
@@
 jumper to select ignition polarity
 $Comp
-L +5V_SWITCHED #PWR?
+L +5V_SWITCHED #PWR065
 U 1 1 4E940836
 P 4750 3250
-F 0 "#PWR?" H 4750 3200 20  0001 C CNN
+F 0 "#PWR065" H 4750 3200 20  0001 C CNN
 F 1 "+5V_SWITCHED" H 4750 3350 30  0000 C CNN
 	1    4750 3250
@@
 $EndComp
 $Comp
-L GND #PWR?
+L GND #PWR066
 U 1 1 4E94061F
 P 4750 4400
-F 0 "#PWR?" H 4750 4400 30  0001 C CNN
+F 0 "#PWR066" H 4750 4400 30  0001 C CNN
 F 1 "GND" H 4750 4330 30  0001 C CNN
 	1    4750 4400
@@
 $EndComp
 $Comp
-L GND #PWR?
+L GND #PWR067
 U 1 1 4E94057E
 P 3100 4050
-F 0 "#PWR?" H 3100 4050 30  0001 C CNN
+F 0 "#PWR067" H 3100 4050 30  0001 C CNN
 F 1 "GND" H 3100 3980 30  0001 C CNN
 	1    3100 4050
@@
 $EndComp
 $Comp
-L CONN_3 K?
+L CONN_3 K2
 U 1 1 4E940542
 P 3200 2850
-F 0 "K?" V 3150 2850 50  0000 C CNN
-F 1 "CONN_3" V 3250 2850 40  0000 C CNN
+F 0 "K2" V 3150 2850 50  0000 C CNN
+F 1 "jumper" V 3250 2850 40  0000 C CNN
 	1    3200 2850
 	0    -1   -1   0
 $EndComp
 $Comp
-L GND #PWR?
+L GND #PWR068
 U 1 1 4E940525
 P 2200 4450
-F 0 "#PWR?" H 2200 4450 30  0001 C CNN
+F 0 "#PWR068" H 2200 4450 30  0001 C CNN
 F 1 "GND" H 2200 4380 30  0001 C CNN
 	1    2200 4450
@@
 $EndComp
 $Comp
-L GND #PWR?
+L GND #PWR069
 U 1 1 4E940520
 P 1950 4450
-F 0 "#PWR?" H 1950 4450 30  0001 C CNN
+F 0 "#PWR069" H 1950 4450 30  0001 C CNN
 F 1 "GND" H 1950 4380 30  0001 C CNN
 	1    1950 4450
@@
 PT3
 $Comp
-L C C?
+L C C30
 U 1 1 4E940494
 P 4750 4100
-F 0 "C?" H 4800 4200 50  0000 L CNN
-F 1 "C" H 4800 4000 50  0000 L CNN
+F 0 "C30" H 4600 4200 50  0000 L CNN
+F 1 "0.1uF" H 4500 4000 50  0000 L CNN
 	1    4750 4100
 	-1   0    0    1
 $EndComp
 $Comp
-L R R?
+L R R37
 U 1 1 4E94048E
 P 2200 4100
-F 0 "R?" V 2280 4100 50  0000 C CNN
-F 1 "R" V 2200 4100 50  0000 C CNN
+F 0 "R37" V 2280 4100 50  0000 C CNN
+F 1 "100K" V 2200 4100 50  0000 C CNN
 	1    2200 4100
 	1    0    0    -1
 $EndComp
 $Comp
-L R R?
+L R R36
 U 1 1 4E94048B
 P 1950 4100
-F 0 "R?" V 2030 4100 50  0000 C CNN
-F 1 "R" V 1950 4100 50  0000 C CNN
+F 0 "R36" V 2030 4100 50  0000 C CNN
+F 1 "100K" V 1950 4100 50  0000 C CNN
 	1    1950 4100
 	1    0    0    -1
 $EndComp
 $Comp
-L R R?
+L R R34
 U 1 1 4E940487
 P 2650 3350
-F 0 "R?" V 2730 3350 50  0000 C CNN
-F 1 "R" V 2650 3350 50  0000 C CNN
+F 0 "R34" V 2730 3350 50  0000 C CNN
+F 1 "1K" V 2650 3350 50  0000 C CNN
 	1    2650 3350
 	0    1    1    0
 $EndComp
 $Comp
-L R R?
+L R R35
 U 1 1 4E940485
 P 2650 3650
-F 0 "R?" V 2730 3650 50  0000 C CNN
-F 1 "R" V 2650 3650 50  0000 C CNN
+F 0 "R35" V 2730 3650 50  0000 C CNN
+F 1 "1K" V 2650 3650 50  0000 C CNN
 	1    2650 3650
 	0    1    1    0
 $EndComp
 $Comp
-L NC7WZ86K8X U?
+L NC7WZ86K8X U5
 U 1 1 4E940421
 P 4050 3700
-F 0 "U?" H 4050 3450 60  0000 C CNN
+F 0 "U5" H 4050 3450 60  0000 C CNN
 F 1 "NC7WZ86K8X" H 4050 3950 60  0000 C CNN
 	1    4050 3700
@@
 Text HLabel 8200 4100 2    60   Input ~ 0
 IGNITER_2_3
-$Comp
-L HCURGND #PWR?
-U 1 1 4E93D675
-P 8900 5850
-F 0 "#PWR?" H 8900 5850 40  0001 C CNN
-F 1 "HCURGND" H 8900 5780 40  0000 C CNN
-	1    8900 5850
-	-1   0    0    -1
-$EndComp
 NoConn ~ 7150 5100
 NoConn ~ 7150 4900
 $Comp
-L GND #PWR?
+L GND #PWR070
 U 1 1 4E93D674
 P 7250 5850
-F 0 "#PWR?" H 7250 5850 30  0001 C CNN
+F 0 "#PWR070" H 7250 5850 30  0001 C CNN
 F 1 "GND" H 7250 5780 30  0001 C CNN
 	1    7250 5850
@@
 $EndComp
 $Comp
-L CAPAPOL C?
+L CAPAPOL C31
 U 1 1 4E93D673
 P 6600 5300
-F 0 "C?" H 6650 5400 50  0000 L CNN
+F 0 "C31" H 6650 5400 50  0000 L CNN
 F 1 "1uF" H 6650 5200 50  0000 L CNN
 	1    6600 5300
@@
 $EndComp
 $Comp
-L C C?
+L C C32
 U 1 1 4E93D672
 P 6950 5300
-F 0 "C?" H 7000 5400 50  0000 L CNN
+F 0 "C32" H 7000 5400 50  0000 L CNN
 F 1 "100nf" H 7000 5200 50  0000 L CNN
 	1    6950 5300
@@
 $EndComp
 $Comp
-L R R?
+L R R39
 U 1 1 4E93D671
 P 6500 4400
-F 0 "R?" V 6580 4400 50  0000 C CNN
+F 0 "R39" V 6580 4400 50  0000 C CNN
 F 1 "1k" V 6500 4400 50  0000 C CNN
 	1    6500 4400
@@
 $EndComp
 $Comp
-L R R?
+L R R40
 U 1 1 4E93D670
 P 6500 4600
-F 0 "R?" V 6580 4600 50  0000 C CNN
+F 0 "R40" V 6580 4600 50  0000 C CNN
 F 1 "1k" V 6500 4600 50  0000 C CNN
 	1    6500 4600
@@
 $EndComp
 $Comp
-L VB325SP U?
+L VB325SP U6
 U 1 1 4E93D66F
 P 7900 4900
-F 0 "U?" H 7900 4600 60  0000 C CNN
+F 0 "U6" H 7900 4600 60  0000 C CNN
 F 1 "VB325SP" H 8300 5300 60  0000 C CNN
 	1    7900 4900
@@
 $EndComp
 $Comp
-L VB325SP U?
+L VB325SP U4
 U 1 1 4E939C23
 P 8000 2500
-F 0 "U?" H 8000 2200 60  0000 C CNN
+F 0 "U4" H 8000 2200 60  0000 C CNN
 F 1 "VB325SP" H 8400 2900 60  0000 C CNN
 	1    8000 2500
@@
 $EndComp
 $Comp
-L R R?
+L R R33
 U 1 1 4E939C22
 P 6600 2200
-F 0 "R?" V 6680 2200 50  0000 C CNN
+F 0 "R33" V 6680 2200 50  0000 C CNN
 F 1 "1k" V 6600 2200 50  0000 C CNN
 	1    6600 2200
@@
 $EndComp
 $Comp
-L R R?
+L R R32
 U 1 1 4E939C21
 P 6600 2000
-F 0 "R?" V 6680 2000 50  0000 C CNN
+F 0 "R32" V 6680 2000 50  0000 C CNN
 F 1 "1k" V 6600 2000 50  0000 C CNN
 	1    6600 2000
@@
 $EndComp
 $Comp
-L C C?
+L C C29
 U 1 1 4E939C20
 P 7050 2900
-F 0 "C?" H 7100 3000 50  0000 L CNN
+F 0 "C29" H 7100 3000 50  0000 L CNN
 F 1 "100nf" H 7100 2800 50  0000 L CNN
 	1    7050 2900
@@
 $EndComp
 $Comp
-L CAPAPOL C?
+L CAPAPOL C28
 U 1 1 4E939C1F
 P 6700 2900
-F 0 "C?" H 6750 3000 50  0000 L CNN
+F 0 "C28" H 6750 3000 50  0000 L CNN
 F 1 "1uF" H 6750 2800 50  0000 L CNN
 	1    6700 2900
@@
 $EndComp
 $Comp
-L GND #PWR?
+L GND #PWR071
 U 1 1 4E939C1E
 P 7350 3450
-F 0 "#PWR?" H 7350 3450 30  0001 C CNN
+F 0 "#PWR071" H 7350 3450 30  0001 C CNN
 F 1 "GND" H 7350 3380 30  0001 C CNN
 	1    7350 3450
@@
 NoConn ~ 7250 2500
 NoConn ~ 7250 2700
-$Comp
-L HCURGND #PWR?
-U 1 1 4E939C1D
-P 9000 3450
-F 0 "#PWR?" H 9000 3450 40  0001 C CNN
-F 1 "HCURGND" H 9000 3380 40  0000 C CNN
-	1    9000 3450
-	-1   0    0    -1
-$EndComp
 Text HLabel 8200 1700 2    60   Input ~ 0
 IGNITER_1_4

Commit message: add test points on critical output, resolve all kind of DRC issue, generate a netlist
Parts:
- added W3, W4: TEST, symbol TEST
Connections:
- wire segments 82 -> 90
Changed lines of the file:
@@
-EESchema Schematic File Version 2  date 02/01/2012 14:25:41
+EESchema Schematic File Version 2  date 03/01/2012 09:04:48
 LIBS:power
 LIBS:device
@@
 Sheet 6 12
 Title "ignition module"
-Date "2 jan 2012"
+Date "3 jan 2012"
 Rev "0.01"
 Comp "diyefi.org"
@@
 Comment4 ""
 $EndDescr
+$Comp
+L GND #PWR68
+U 1 1 4F01C2F1
+P 5800 4200
+F 0 "#PWR68" H 5800 4200 30  0001 C CNN
+F 1 "GND" H 5800 4130 30  0001 C CNN
+	1    5800 4200
+	1    0    0    -1
+$EndComp
+Wire Wire Line
+	5800 4200 5800 3950
+Wire Wire Line
+	5800 3950 5650 3950
+Wire Wire Line
+	5800 3450 5800 3200
+Wire Wire Line
+	5800 3200 5650 3200
 Wire Wire Line
 	8900 5850 8900 4800
-$Comp
-L IGNGND #PWR059
-U 1 1 4EFDEBD7
-P 8900 5850
-F 0 "#PWR059" H 8900 5850 40  0001 C CNN
-F 1 "IGNGND" H 8900 5780 40  0000 C CNN
-	1    8900 5850
-	1    0    0    -1
-$EndComp
-$Comp
-L IGNGND #PWR060
-U 1 1 4EFDEBD2
-P 9000 3450
-F 0 "#PWR060" H 9000 3450 40  0001 C CNN
-F 1 "IGNGND" H 9000 3380 40  0000 C CNN
-	1    9000 3450
-	1    0    0    -1
-$EndComp
 Connection ~ 8000 1700
 Wire Wire Line
@@
 Connection ~ 7900 4100
 Wire Wire Line
-	8200 4100 7650 4100
+	7650 4100 8200 4100
 Wire Wire Line
 	7200 1700 7350 1700
@@
 Connection ~ 3100 3850
 Wire Wire Line
-	3100 4050 3100 3200
+	3100 3200 3100 4050
 Wire Wire Line
 	3500 3550 3200 3550
@@
 	2200 3850 2200 3350
 Wire Wire Line
-	2400 3350 1750 3350
+	1750 3350 2400 3350
 Wire Wire Line
 	3500 3650 2900 3650
@@
 	7050 3350 7050 3100
 Wire Wire Line
-	6700 2400 6700 2700
-Wire Wire Line
-	8750 2700 8750 3350
+	6700 2700 6700 2400
+Wire Wire Line
+	8750 3350 8750 2700
 Connection ~ 9000 2600
 Wire Wire Line
@@
 Connection ~ 7050 2400
 Wire Wire Line
-	6700 3350 6700 3100
+	6700 3100 6700 3350
 Connection ~ 7050 3350
 Wire Wire Line
-	7050 2700 7050 2400
+	7050 2400 7050 2700
 Wire Wire Line
 	7350 3350 7350 3450
@@
 	7250 5750 7250 5850
 Wire Wire Line
-	6950 4800 6950 5100
+	6950 5100 6950 4800
 Connection ~ 6950 5750
 Wire Wire Line
@@
 	8650 5100 8650 5750
 Wire Wire Line
-	6600 5100 6600 4800
+	6600 4800 6600 5100
 Wire Wire Line
 	6950 5750 6950 5500
@@
 	4900 3350 2900 3350
 Wire Wire Line
-	2400 3650 1750 3650
+	1750 3650 2400 3650
 Wire Wire Line
 	1950 3850 1950 3650
@@
 	5900 2400 5900 2250
 Wire Wire Line
-	8200 1700 7750 1700
+	7750 1700 8200 1700
 Wire Wire Line
 	6250 3900 6250 4100
@@
 Wire Wire Line
 	7900 4350 7900 4100
+Wire Wire Line
+	5250 3200 5100 3200
+Wire Wire Line
+	5100 3200 5100 3650
+Connection ~ 5100 3650
+Wire Wire Line
+	5250 3950 5100 3950
+Wire Wire Line
+	5100 3950 5100 4600
+Connection ~ 5100 4600
+$Comp
+L TEST W4
+U 1 1 4F01C2DB
+P 5450 3950
+F 0 "W4" H 5450 4010 40  0000 C CNN
+F 1 "TEST" H 5450 3880 40  0000 C CNN
+	1    5450 3950
+	1    0    0    -1
+$EndComp
+$Comp
+L GND #PWR63
+U 1 1 4F01C251
+P 5800 3450
+F 0 "#PWR63" H 5800 3450 30  0001 C CNN
+F 1 "GND" H 5800 3380 30  0001 C CNN
+	1    5800 3450
+	1    0    0    -1
+$EndComp
+$Comp
+L TEST W3
+U 1 1 4F01C234
+P 5450 3200
+F 0 "W3" H 5450 3260 40  0000 C CNN
+F 1 "TEST" H 5450 3130 40  0000 C CNN
+	1    5450 3200
+	1    0    0    -1
+$EndComp
+$Comp
+L IGNGND #PWR74
+U 1 1 4EFDEBD7
+P 8900 5850
+F 0 "#PWR74" H 8900 5850 40  0001 C CNN
+F 1 "IGNGND" H 8900 5780 40  0000 C CNN
+	1    8900 5850
+	1    0    0    -1
+$EndComp
+$Comp
+L IGNGND #PWR65
+U 1 1 4EFDEBD2
+P 9000 3450
+F 0 "#PWR65" H 9000 3450 40  0001 C CNN
+F 1 "IGNGND" H 9000 3380 40  0000 C CNN
+	1    9000 3450
+	1    0    0    -1
+$EndComp
 $Comp
 L R R38
@@
 $EndComp
 $Comp
-L +12V_SWITCHED #PWR061
+L +12V_SWITCHED #PWR66
 U 1 1 4E95AA72
 P 6250 3900
-F 0 "#PWR061" H 6250 3850 20  0001 C CNN
+F 0 "#PWR66" H 6250 3850 20  0001 C CNN
 F 1 "+12V_SWITCHED" H 6250 4000 30  0000 C CNN
 	1    6250 3900
@@
 $EndComp
 $Comp
-L +12V_SWITCHED #PWR062
+L +12V_SWITCHED #PWR60
 U 1 1 4E95AA35
 P 6350 1500
-F 0 "#PWR062" H 6350 1450 20  0001 C CNN
+F 0 "#PWR60" H 6350 1450 20  0001 C CNN
 F 1 "+12V_SWITCHED" H 6350 1600 30  0000 C CNN
 	1    6350 1500
@@
 $EndComp
 $Comp
-L +5V_SWITCHED #PWR063
+L +5V_SWITCHED #PWR72
 U 1 1 4E9456A3
 P 5900 4500
-F 0 "#PWR063" H 5900 4450 20  0001 C CNN
+F 0 "#PWR72" H 5900 4450 20  0001 C CNN
 F 1 "+5V_SWITCHED" H 5900 4600 30  0000 C CNN
 	1    5900 4500
@@
 $EndComp
 $Comp
-L +5V_SWITCHED #PWR064
+L +5V_SWITCHED #PWR61
 U 1 1 4E94565D
 P 5900 2250
-F 0 "#PWR064" H 5900 2200 20  0001 C CNN
+F 0 "#PWR61" H 5900 2200 20  0001 C CNN
 F 1 "+5V_SWITCHED" H 5900 2350 30  0000 C CNN
 	1    5900 2250
@@
 jumper to select ignition polarity
 $Comp
-L +5V_SWITCHED #PWR065
+L +5V_SWITCHED #PWR62
 U 1 1 4E940836
 P 4750 3250
-F 0 "#PWR065" H 4750 3200 20  0001 C CNN
+F 0 "#PWR62" H 4750 3200 20  0001 C CNN
 F 1 "+5V_SWITCHED" H 4750 3350 30  0000 C CNN
 	1    4750 3250
@@
 $EndComp
 $Comp
-L GND #PWR066
+L GND #PWR69
 U 1 1 4E94061F
 P 4750 4400
-F 0 "#PWR066" H 4750 4400 30  0001 C CNN
+F 0 "#PWR69" H 4750 4400 30  0001 C CNN
 F 1 "GND" H 4750 4330 30  0001 C CNN
 	1    4750 4400
@@
 $EndComp
 $Comp
-L GND #PWR067
+L GND #PWR67
 U 1 1 4E94057E
 P 3100 4050
-F 0 "#PWR067" H 3100 4050 30  0001 C CNN
+F 0 "#PWR67" H 3100 4050 30  0001 C CNN
 F 1 "GND" H 3100 3980 30  0001 C CNN
 	1    3100 4050
@@
 $EndComp
 $Comp
-L GND #PWR068
+L GND #PWR71
 U 1 1 4E940525
 P 2200 4450
-F 0 "#PWR068" H 2200 4450 30  0001 C CNN
+F 0 "#PWR71" H 2200 4450 30  0001 C CNN
 F 1 "GND" H 2200 4380 30  0001 C CNN
 	1    2200 4450
@@
 $EndComp
 $Comp
-L GND #PWR069
+L GND #PWR70
 U 1 1 4E940520
 P 1950 4450
-F 0 "#PWR069" H 1950 4450 30  0001 C CNN
+F 0 "#PWR70" H 1950 4450 30  0001 C CNN
 F 1 "GND" H 1950 4380 30  0001 C CNN
 	1    1950 4450
@@
 NoConn ~ 7150 4900
 $Comp
-L GND #PWR070
+L GND #PWR73
 U 1 1 4E93D674
 P 7250 5850
-F 0 "#PWR070" H 7250 5850 30  0001 C CNN
+F 0 "#PWR73" H 7250 5850 30  0001 C CNN
 F 1 "GND" H 7250 5780 30  0001 C CNN
 	1    7250 5850
@@
 $EndComp
 $Comp
-L GND #PWR071
+L GND #PWR64
 U 1 1 4E939C1E
 P 7350 3450
-F 0 "#PWR071" H 7350 3450 30  0001 C CNN
+F 0 "#PWR64" H 7350 3450 30  0001 C CNN
 F 1 "GND" H 7350 3380 30  0001 C CNN
 	1    7350 3450

Commit message: add missing diodes, re-generate netlist, assign all footprints, ready to layout
Parts:
- removed U5: NC7WZ86K8X, symbol NC7WZ86K8X
- added U5: 74LS86_MW, symbol 74LS86_MW
- renumbered D14 to D15, D15 to D16
Changed lines of the file:
@@
-EESchema Schematic File Version 2  date 03/01/2012 09:04:48
+EESchema Schematic File Version 2  date 12/01/2012 20:05:35
 LIBS:power
 LIBS:device
@@
 Sheet 6 12
 Title "ignition module"
-Date "3 jan 2012"
+Date "12 jan 2012"
 Rev "0.01"
 Comp "diyefi.org"
@@
 $EndDescr
 $Comp
+L 74LS86_MW U5
+U 1 1 4F07A6A8
+P 4050 3700
+F 0 "U5" H 4050 3450 60  0000 C CNN
+F 1 "74LS86_MW" H 4050 3950 60  0000 C CNN
+	1    4050 3700
+	1    0    0    -1
+$EndComp
+$Comp
 L GND #PWR68
 U 1 1 4F01C2F1
@@
 $EndComp
 $Comp
-L LED D15
+L LED D16
 U 1 1 4E95AA73
 P 7450 4100
-F 0 "D15" H 7450 4200 50  0000 C CNN
+F 0 "D16" H 7450 4200 50  0000 C CNN
 F 1 "LED" H 7450 4000 50  0000 C CNN
 	1    7450 4100
@@
 $EndComp
 $Comp
-L LED D14
+L LED D15
 U 1 1 4E95AA36
 P 7550 1700
-F 0 "D14" H 7550 1800 50  0000 C CNN
+F 0 "D15" H 7550 1800 50  0000 C CNN
 F 1 "LED" H 7550 1600 50  0000 C CNN
 	1    7550 1700
@@
 	0    1    1    0
 $EndComp
-$Comp
-L NC7WZ86K8X U5
-U 1 1 4E940421
-P 4050 3700
-F 0 "U5" H 4050 3450 60  0000 C CNN
-F 1 "NC7WZ86K8X" H 4050 3950 60  0000 C CNN
-	1    4050 3700
-	1    0    0    -1
-$EndComp
 Text HLabel 8200 4100 2    60   Input ~ 0
