File: design/U_Igniter Outputs.sch (KiCad schematic (older format))
At the start: 23 parts, among them K2 jumper, U4 VB325SP, U5 74LS86_MW, U6 VB325SP

Commit message: revise schema according to Jaguar & Ravage project, eliminate as many errors as possible which were inherited from Puma board. Remove VSS interface, narrow band O2 interface, AC relay output, AC signal input. Make fuel injection configurable which can be batch fired or semi sequential fired
Parts:
- removed W3, W4: TEST, symbol TEST
- added D18, D19: 1N4148, symbol DIODE
Connections:
- wire segments 90 -> 82
Other:
- moved on the sheet: C31, C32, D15, D16, R31, R38, R39, R40, U6

Commit message: make new footprint for screw connector, redesign ignition gnd & all lowside gnd
Parts:
- K1: renamed from K2; value jumper -> Polarity
Changed lines of the file:
@@
-EESchema Schematic File Version 2  date 02/02/2012 10:58:16
+EESchema Schematic File Version 2  date 07/02/2012 00:44:28
 LIBS:power
 LIBS:device
@@
 Sheet 6 10
 Title "ignition module"
-Date "2 feb 2012"
+Date "6 feb 2012"
 Rev "0.01"
 Comp "diyefi.org"
@@
 $EndComp
 $Comp
-L IGNGND #PWR056
+L IGNGND #PWR059
 U 1 1 4EFDEBD7
 P 9000 5850
-F 0 "#PWR056" H 9000 5850 40  0001 C CNN
+F 0 "#PWR059" H 9000 5850 40  0001 C CNN
 F 1 "IGNGND" H 9000 5780 40  0000 C CNN
 	1    9000 5850
@@
 $EndComp
 $Comp
-L IGNGND #PWR057
+L IGNGND #PWR060
 U 1 1 4EFDEBD2
 P 9000 3450
-F 0 "#PWR057" H 9000 3450 40  0001 C CNN
+F 0 "#PWR060" H 9000 3450 40  0001 C CNN
 F 1 "IGNGND" H 9000 3380 40  0000 C CNN
 	1    9000 3450
@@
 $EndComp
 $Comp
-L +12V_SWITCHED #PWR058
+L +12V_SWITCHED #PWR061
 U 1 1 4E95AA72
 P 6350 3900
-F 0 "#PWR058" H 6350 3850 20  0001 C CNN
+F 0 "#PWR061" H 6350 3850 20  0001 C CNN
 F 1 "+12V_SWITCHED" H 6350 4000 30  0000 C CNN
 	1    6350 3900
@@
 $EndComp
 $Comp
-L +12V_SWITCHED #PWR059
+L +12V_SWITCHED #PWR062
 U 1 1 4E95AA35
 P 6350 1500
-F 0 "#PWR059" H 6350 1450 20  0001 C CNN
+F 0 "#PWR062" H 6350 1450 20  0001 C CNN
 F 1 "+12V_SWITCHED" H 6350 1600 30  0000 C CNN
 	1    6350 1500
@@
 $EndComp
 $Comp
-L +5V_SWITCHED #PWR060
+L +5V_SWITCHED #PWR063
 U 1 1 4E9456A3
 P 6000 4500
-F 0 "#PWR060" H 6000 4450 20  0001 C CNN
+F 0 "#PWR063" H 6000 4450 20  0001 C CNN
 F 1 "+5V_SWITCHED" H 6000 4600 30  0000 C CNN
 	1    6000 4500
@@
 $EndComp
 $Comp
-L +5V_SWITCHED #PWR061
+L +5V_SWITCHED #PWR064
 U 1 1 4E94565D
 P 5900 2250
-F 0 "#PWR061" H 5900 2200 20  0001 C CNN
+F 0 "#PWR064" H 5900 2200 20  0001 C CNN
 F 1 "+5V_SWITCHED" H 5900 2350 30  0000 C CNN
 	1    5900 2250
@@
 jumper to select ignition polarity
 $Comp
-L +5V_SWITCHED #PWR062
+L +5V_SWITCHED #PWR065
 U 1 1 4E940836
 P 4750 3250
-F 0 "#PWR062" H 4750 3200 20  0001 C CNN
+F 0 "#PWR065" H 4750 3200 20  0001 C CNN
 F 1 "+5V_SWITCHED" H 4750 3350 30  0000 C CNN
 	1    4750 3250
@@
 $EndComp
 $Comp
-L GND #PWR063
+L GND #PWR066
 U 1 1 4E94061F
 P 4750 4400
-F 0 "#PWR063" H 4750 4400 30  0001 C CNN
+F 0 "#PWR066" H 4750 4400 30  0001 C CNN
 F 1 "GND" H 4750 4330 30  0001 C CNN
 	1    4750 4400
@@
 $EndComp
 $Comp
-L GND #PWR064
+L GND #PWR067
 U 1 1 4E94057E
 P 3100 4050
-F 0 "#PWR064" H 3100 4050 30  0001 C CNN
+F 0 "#PWR067" H 3100 4050 30  0001 C CNN
 F 1 "GND" H 3100 3980 30  0001 C CNN
 	1    3100 4050
@@
 $EndComp
 $Comp
-L CONN_3 K2
+L CONN_3 K1
 U 1 1 4E940542
 P 3200 2850
-F 0 "K2" V 3150 2850 50  0000 C CNN
-F 1 "jumper" V 3250 2850 40  0000 C CNN
+F 0 "K1" V 3150 2850 50  0000 C CNN
+F 1 "Polarity" V 3250 2850 40  0000 C CNN
 	1    3200 2850
 	0    -1   -1   0
 $EndComp
 $Comp
-L GND #PWR065
+L GND #PWR068
 U 1 1 4E940525
 P 2200 4450
-F 0 "#PWR065" H 2200 4450 30  0001 C CNN
+F 0 "#PWR068" H 2200 4450 30  0001 C CNN
 F 1 "GND" H 2200 4380 30  0001 C CNN
 	1    2200 4450
@@
 $EndComp
 $Comp
-L GND #PWR066
+L GND #PWR069
 U 1 1 4E940520
 P 1950 4450
-F 0 "#PWR066" H 1950 4450 30  0001 C CNN
+F 0 "#PWR069" H 1950 4450 30  0001 C CNN
 F 1 "GND" H 1950 4380 30  0001 C CNN
 	1    1950 4450
@@
 NoConn ~ 7250 4900
 $Comp
-L GND #PWR067
+L GND #PWR070
 U 1 1 4E93D674
 P 7350 5850
-F 0 "#PWR067" H 7350 5850 30  0001 C CNN
+F 0 "#PWR070" H 7350 5850 30  0001 C CNN
 F 1 "GND" H 7350 5780 30  0001 C CNN
 	1    7350 5850
@@
 $EndComp
 $Comp
-L GND #PWR068
+L GND #PWR071
 U 1 1 4E939C1E
 P 7350 3450
-F 0 "#PWR068" H 7350 3450 30  0001 C CNN
+F 0 "#PWR071" H 7350 3450 30  0001 C CNN
 F 1 "GND" H 7350 3380 30  0001 C CNN
 	1    7350 3450
