File: design/VR Interfaces.sch (KiCad schematic (older format))
At the start: 7 parts, among them U8 MAX9924

Commit message: revise schema according to Jaguar & Ravage project, eliminate as many errors as possible which were inherited from Puma board. Remove VSS interface, narrow band O2 interface, AC relay output, AC signal input. Make fuel injection configurable which can be batch fired or semi sequential fired
Parts:
- removed W6: TEST, symbol TEST
- added C52: 1uF, symbol C
- added C53: 10nF, symbol C
- added D30: LED, symbol LED
- added R28: 5k, symbol R
- added R29: ??, symbol R
Connections:
- wire segments 25 -> 23
Other:
- moved on the sheet: C38, C45, R63, R64, R65
Changed lines of the file:
@@
-EESchema Schematic File Version 2  date 29/01/2012 19:39:37
+EESchema Schematic File Version 2  date 02/02/2012 00:51:37
 LIBS:power
 LIBS:device
@@
 EELAYER END
 $Descr A4 11700 8267
-Sheet 10 12
+Sheet 9 10
 Title "VR interface"
-Date "24 jan 2012"
+Date "1 feb 2012"
 Rev "0.01"
 Comp "diyefi.org"
@@
 Comment4 ""
 $EndDescr
-Connection ~ 4200 3750
-Connection ~ 4200 3350
-Wire Wire Line
-	4100 3350 4550 3350
-Wire Wire Line
-	6600 4250 6600 3550
-Wire Wire Line
-	6600 4150 4550 4150
-Connection ~ 7300 3900
-Wire Wire Line
-	7300 3750 7300 3900
-Wire Wire Line
-	4550 4150 4550 3900
-Wire Wire Line
-	3450 3750 3600 3750
-Wire Wire Line
-	4550 3350 4550 3600
-Wire Wire Line
-	4550 3600 4700 3600
-Wire Wire Line
-	4550 3700 4550 3750
-Wire Wire Line
-	4550 3700 4700 3700
-Connection ~ 7050 3900
-Wire Wire Line
-	7050 3800 7050 3900
-Connection ~ 6600 4000
-Wire Wire Line
-	6200 3700 6600 3700
+Wire Wire Line
+	7200 3900 7500 3900
+Wire Wire Line
+	7500 3900 7500 4150
+Wire Wire Line
+	6500 4150 6500 3700
+Wire Wire Line
+	6500 3700 7200 3700
+Connection ~ 6850 3150
+Wire Wire Line
+	7200 3150 6300 3150
+Wire Wire Line
+	4700 3900 4550 3900
+Wire Wire Line
+	4550 3900 4550 4150
+Wire Wire Line
+	4700 3700 4150 3700
+Wire Wire Line
+	4150 3300 4500 3300
+Connection ~ 4550 4000
+Connection ~ 6300 4000
+Wire Wire Line
+	6200 4000 6300 4000
+Connection ~ 7200 3150
+Wire Wire Line
+	3400 3300 3650 3300
+Connection ~ 6500 3150
+Wire Wire Line
+	6300 3150 6300 3600
+Wire Wire Line
+	6300 3600 6200 3600
 Wire Wire Line
 	4700 4000 4550 4000
 Wire Wire Line
-	6200 3600 6300 3600
-Wire Wire Line
-	6300 3600 6300 3150
-Wire Wire Line
-	4550 3900 4700 3900
-Connection ~ 4550 4000
-Wire Wire Line
-	6600 4000 6200 4000
-Connection ~ 6600 3700
-Wire Wire Line
-	7450 3900 6200 3900
-Wire Wire Line
-	6300 3150 7050 3150
-Wire Wire Line
-	7050 3150 7050 3300
-Connection ~ 6600 3150
-Wire Wire Line
-	4550 3750 4100 3750
-Wire Wire Line
-	3600 3350 3450 3350
-Connection ~ 6600 4150
-Wire Wire Line
-	7300 3350 7300 3250
-Wire Wire Line
-	7300 3250 7500 3250
-Wire Wire Line
-	7500 3250 7500 3400
-$Comp
-L GND #PWR0107
+	4550 4150 6300 4150
+Connection ~ 4250 3300
+Connection ~ 4250 3700
+Wire Wire Line
+	6200 3700 6300 3700
+Wire Wire Line
+	6300 3700 6300 4250
+Connection ~ 6300 4150
+Connection ~ 3550 3300
+Wire Wire Line
+	3400 3800 3650 3800
+Wire Wire Line
+	3650 3800 3650 3700
+Connection ~ 3550 3800
+Wire Wire Line
+	4500 3300 4500 3600
+Wire Wire Line
+	4500 3600 4700 3600
+Connection ~ 6500 3900
+Wire Wire Line
+	7100 4150 7000 4150
+Wire Wire Line
+	6700 3900 6200 3900
+$Comp
+L LED D30
+U 1 1 4F296C18
+P 7300 4150
+F 0 "D30" H 7300 4250 50  0000 C CNN
+F 1 "LED" H 7300 4050 50  0000 C CNN
+	1    7300 4150
+	-1   0    0    1
+$EndComp
+$Comp
+L R R29
+U 1 1 4F296BDB
+P 6750 4150
+F 0 "R29" V 6830 4150 50  0000 C CNN
+F 1 "??" V 6750 4150 50  0000 C CNN
+	1    6750 4150
+	0    1    1    0
+$EndComp
+$Comp
+L +5V_SWITCHED #PWR084
+U 1 1 4F296B6A
+P 7500 3900
+F 0 "#PWR084" H 7500 3850 20  0001 C CNN
+F 1 "+5V_SWITCHED" H 7500 4000 30  0000 C CNN
+	1    7500 3900
+	1    0    0    -1
+$EndComp
+$Comp
+L R R28
+U 1 1 4F296984
+P 3550 3550
+F 0 "R28" V 3630 3550 50  0000 C CNN
+F 1 "5k" V 3550 3550 50  0000 C CNN
+	1    3550 3550
+	1    0    0    -1
+$EndComp
+$Comp
+L GND #PWR085
+U 1 1 4F296901
+P 6500 3550
+F 0 "#PWR085" H 6500 3550 30  0001 C CNN
+F 1 "GND" H 6500 3480 30  0001 C CNN
+	1    6500 3550
+	1    0    0    -1
+$EndComp
+$Comp
+L GND #PWR086
+U 1 1 4F296882
+P 7200 3550
+F 0 "#PWR086" H 7200 3550 30  0001 C CNN
+F 1 "GND" H 7200 3480 30  0001 C CNN
+	1    7200 3550
+	1    0    0    -1
+$EndComp
+$Comp
+L GND #PWR087
+U 1 1 4F29687C
+P 6850 3550
+F 0 "#PWR087" H 6850 3550 30  0001 C CNN
+F 1 "GND" H 6850 3480 30  0001 C CNN
+	1    6850 3550
+	1    0    0    -1
+$EndComp
+$Comp
+L C C53
+U 1 1 4F296777
+P 7200 3350
+F 0 "C53" H 7250 3450 50  0000 L CNN
+F 1 "10nF" H 7250 3250 50  0000 L CNN
+	1    7200 3350
+	1    0    0    -1
+$EndComp
+$Comp
+L C C52
+U 1 1 4F296773
+P 6850 3350
+F 0 "C52" H 6900 3450 50  0000 L CNN
+F 1 "1uF" H 6900 3250 50  0000 L CNN
+	1    6850 3350
+	1    0    0    -1
+$EndComp
+$Comp
+L GND #PWR088
 U 1 1 4F193950
-P 6600 4250
-F 0 "#PWR0107" H 6600 4250 30  0001 C CNN
-F 1 "GND" H 6600 4180 30  0001 C CNN
-	1    6600 4250
+P 6300 4250
+F 0 "#PWR088" H 6300 4250 30  0001 C CNN
+F 1 "GND" H 6300 4180 30  0001 C CNN
+	1    6300 4250
 	1    0    0    -1
 $EndComp
@@
 L C C38
 U 1 1 4F19371B
-P 6600 3350
-F 0 "C38" H 6650 3450 50  0000 L CNN
-F 1 "0.1uF" H 6650 3250 50  0000 L CNN
-	1    6600 3350
+P 6500 3350
+F 0 "C38" H 6550 3450 50  0000 L CNN
+F 1 "0.1uF" H 6550 3250 50  0000 L CNN
+	1    6500 3350
 	1    0    0    -1
 $EndComp
@@
 L R R64
 U 1 1 4F19371A
-P 7050 3550
-F 0 "R64" V 7130 3550 50  0000 C CNN
-F 1 "10k" V 7050 3550 50  0000 C CNN
-	1    7050 3550
-	1    0    0    -1
+P 6950 3900
+F 0 "R64" V 7030 3900 50  0000 C CNN
+F 1 "10k" V 6950 3900 50  0000 C CNN
+	1    6950 3900
+	0    1    1    0
 $EndComp
 $Comp
 L C C45
 U 1 1 4F193719
-P 4200 3550
-F 0 "C45" H 4250 3650 50  0000 L CNN
-F 1 "1nF" H 4250 3450 50  0000 L CNN
-	1    4200 3550
+P 4250 3500
+F 0 "C45" H 4300 3600 50  0000 L CNN
+F 1 "1nF" H 4300 3400 50  0000 L CNN
+	1    4250 3500
 	1    0    0    -1
 $EndComp
@@
 L R R65
 U 1 1 4F193718
-P 3850 3750
-F 0 "R65" V 3930 3750 50  0000 C CNN
-F 1 "10k" V 3850 3750 50  0000 C CNN
-	1    3850 3750
+P 3900 3700
+F 0 "R65" V 3980 3700 50  0000 C CNN
+F 1 "10k" V 3900 3700 50  0000 C CNN
+	1    3900 3700
 	0    1    1    0
 $EndComp
@@
 L R R63
 U 1 1 4F193717
-P 3850 3350
-F 0 "R63" V 3930 3350 50  0000 C CNN
-F 1 "10k" V 3850 3350 50  0000 C CNN
-	1    3850 3350
-	0    1    1    0
-$EndComp
-$Comp
-L GND #PWR0108
-U 1 1 4F01BE3E
-P 7500 3400
-F 0 "#PWR0108" H 7500 3400 30  0001 C CNN
-F 1 "GND" H 7500 3330 30  0001 C CNN
-	1    7500 3400
-	1    0    0    -1
-$EndComp
-$Comp
-L TEST W6
-U 1 1 4F01BDF8
-P 7300 3550
-F 0 "W6" H 7300 3610 40  0000 C CNN
-F 1 "TEST" H 7300 3480 40  0000 C CNN
-	1    7300 3550
-	0    -1   -1   0
-$EndComp
-Text HLabel 3450 3750 0    60   Input ~ 0
+P 3900 3300
+F 0 "R63" V 3980 3300 50  0000 C CNN
+F 1 "10k" V 3900 3300 50  0000 C CNN
+	1    3900 3300
+	0    1    1    0
+$EndComp
+Text HLabel 3400 3800 0    60   Input ~ 0
 RPM0-
-Text HLabel 3450 3350 0    60   Input ~ 0
+Text HLabel 3400 3300 0    60   Input ~ 0
 RPM0+
-Text HLabel 7450 3900 2    60   Output ~ 0
+Text HLabel 7200 3700 2    60   Output ~ 0
 PT0
 $Comp
-L +5V_SWITCHED #PWR0109
+L +5V_SWITCHED #PWR089
 U 1 1 4E94109E
 P 6300 3150
-F 0 "#PWR0109" H 6300 3100 20  0001 C CNN
+F 0 "#PWR089" H 6300 3100 20  0001 C CNN
 F 1 "+5V_SWITCHED" H 6300 3250 30  0000 C CNN
 	1    6300 3150

Commit message: revise schema according to DeuceEFI's claim
Parts:
- R29: value ?? -> 2.4K
Other:
- note added: "1 W"
- note added: "1/2 W"
- note added: "1/4 W"
Changed lines of the file:
@@
-EESchema Schematic File Version 2  date 07/02/2012 00:44:28
+EESchema Schematic File Version 2  date 08/02/2012 17:27:58
 LIBS:power
 LIBS:device
@@
 Sheet 9 10
 Title "VR interface"
-Date "6 feb 2012"
+Date "8 feb 2012"
 Rev "0.01"
 Comp "diyefi.org"
@@
 Comment4 ""
 $EndDescr
+Text Notes 6650 4100 0    40   ~ 0
+1/4 W
+Text Notes 3450 3600 1    40   ~ 0
+1 W
+Text Notes 3800 3600 0    40   ~ 0
+1/2 W
+Text Notes 3800 3200 0    40   ~ 0
+1/2 W
 Wire Wire Line
 	7200 3900 7500 3900
@@
 P 6750 4150
 F 0 "R29" V 6830 4150 50  0000 C CNN
-F 1 "??" V 6750 4150 50  0000 C CNN
+F 1 "2.4K" V 6750 4150 50  0000 C CNN
 	1    6750 4150
 	0    1    1    0
