File: design/Core Board.sch (KiCad schematic (older format))
At the start: 31 parts, among them P1 BDM, P2 jumper, P5 CONN_6, SW1 SW_PUSH, U2 MC9S12XDP512, X1 CRYSTAL

Commit message: revise schema according to Jaguar & Ravage project, eliminate as many errors as possible which were inherited from Puma board. Remove VSS interface, narrow band O2 interface, AC relay output, AC signal input. Make fuel injection configurable which can be batch fired or semi sequential fired
Parts:
- removed C24: 104, symbol C
- removed P5: CONN_6, symbol CONN_6
- removed R26, R77, R78, R79, R80: 1.6k, symbol R
- removed SW1: SW_PUSH, symbol SW_PUSH
- added C24, C39, C42, C47: 10uF, symbol CP1
- added C40: 0.22uF, symbol C
- added C41, C44, C49: 0.1uF, symbol C
- added C43, C48: .1uF, C1V7, symbol C
- added C46: 22uF, symbol CP1
- added C50: 47uF, symbol CP1
- added D12: CEL LED, symbol LED
- added D13, D14: 1N5919BG, symbol ZENER
- added R20: 1K, symbol R
- added U10, U9: TLE4275, symbol TLE4275
- C14, C15, C16, C18, C22: value .1uF -> 0.22uF
- C17, C21: value 22pF -> 18pF
- C19: value 3.3nF -> 6.8nF
- C20: value 330pF -> 680pF
- C23: value 100nF -> 0.22uF
- R11: value 3.9K -> 3.3K
- R12: value 10M -> 1M
- R16: value 4.7K -> 10K
- R18: value 100R -> 10K
Connections:
- net labels added: +12V_SWITCHED, ADCGND, IGNGND, LSGND, PB1, PT4, PT5
- net labels removed: AN11, PA0, PA2, PA3, PA4, PA5, PP1, PT6, RXCAN3, TXCAN3
- wire segments 121 -> 120
- no-connect marks 59 -> 69
Other:
- note added: "BootLoader activate"
- note added: "CPU voltage regulator"
- note added: "Power symbols usage\n+12V_SWITCHED come from igniton switch\n+5V_MICRO come from CPU voltage reg \n+5V_SWITCHED come from secondary voltage reg\nLSGND low side ground\nADCGND sensor ground\nIGNGND ignition ground"
- note added: "Switched power regulator"
- note removed: "BootLoader enable"
- note removed: "Van and Vdd must meet each other at the 5v regulator, so digital currents dont mess with the ADC stability.\nAlso, keep an analog ground plane beneath this Van track."
- note removed: "manual reset switch"
- moved on the sheet: C14, C15, C16, C17, C18, C19, C20, C21, C22, C23, P1, P2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

Commit message: make new footprint for screw connector, redesign ignition gnd & all lowside gnd
Parts:
- K2: renamed from P2; value jumper -> Bootldr
Connections:
- net labels removed: IGNGND, LSGND
- wire segments 120 -> 118
Other:
- note added: "ADC and CPU gnd finally\n meet together at regulator"

Commit message: revise schema according to DeuceEFI's claim
Parts:
- C46: value 22uF -> 47uF
- R12: value 1M -> 10M
Other:
- note added: "5.6v/3w"
- note added: "C18 X7R Ceramic"
- note added: "C22 and C40 X7R Ceramic"
- note added: "C24 10v Tantalum\nC15 X7R Ceramic"
- note added: "C39 10v Tantalum\nC16 X7R Ceramic"
- note added: "C42 and C47 are 35v Tantalum capacitors.\nC46 and C50 are 16v Tantalum capacitors."
- note added: "C43, C48, C44 and C49 are 50v X7R Ceramic capacitors."
- note added: "R12 is Optional"
Changed lines of the file:
@@
-EESchema Schematic File Version 2  date 07/02/2012 00:44:28
+EESchema Schematic File Version 2  date 08/02/2012 17:27:58
 LIBS:power
 LIBS:device
@@
 Sheet 3 10
 Title "CPU circuit"
-Date "6 feb 2012"
+Date "8 feb 2012"
 Rev "0.01"
 Comp "diyefi.org"
@@
 Comment4 ""
 $EndDescr
+Text Notes 2000 10100 0    60   ~ 0
+C43, C48, C44 and C49 are 50v X7R Ceramic capacitors.
+Text Notes 2250 10200 0    60   ~ 0
+C42 and C47 are 35v Tantalum capacitors.\nC46 and C50 are 16v Tantalum capacitors.
+Text Notes 5850 9550 0    40   ~ 0
+5.6v/3w
+Text Notes 5850 7650 0    40   ~ 0
+5.6v/3w
+Text Notes 8250 1850 0    60   ~ 0
+C24 10v Tantalum\nC15 X7R Ceramic
+Text Notes 7300 2350 0    60   ~ 0
+C39 10v Tantalum\nC16 X7R Ceramic
+Text Notes 11900 4250 0    60   ~ 0
+C22 and C40 X7R Ceramic
+Text Notes 5650 3400 1    60   ~ 0
+R12 is Optional
+Text Notes 12550 2600 0    60   ~ 0
+C18 X7R Ceramic
 Text Notes 6150 10100 2    60   ~ 0
 ADC and CPU gnd finally\n meet together at regulator
@@
 P 5350 7600
 F 0 "C46" H 5400 7700 50  0000 L CNN
-F 1 "22uF" H 5400 7500 50  0000 L CNN
+F 1 "47uF" H 5400 7500 50  0000 L CNN
 	1    5350 7600
 	1    0    0    -1
@@
 P 5750 3100
 F 0 "R12" V 5830 3100 50  0000 C CNN
-F 1 "1M" V 5750 3100 50  0000 C CNN
+F 1 "10M" V 5750 3100 50  0000 C CNN
 	1    5750 3100
 	1    0    0    -1
@@
 F 1 "18pF" H 5450 3250 50  0000 L CNN
 	1    5400 3350
-	1    0    0    -1
+	-1   0    0    -1
 $EndComp
 $Comp
@@
 F 1 "18pF" H 5450 2750 50  0000 L CNN
 	1    5400 2850
-	1    0    0    -1
+	-1   0    0    -1
 $EndComp
 NoConn ~ 11400 4050

Commit message: some layout work, very dirty
Parts:
- C43, C48: value .1uF -> 0.1uF
Changed lines of the file:
@@
-EESchema Schematic File Version 2  date 08/02/2012 17:27:58
+EESchema Schematic File Version 2  date 06/03/2012 22:16:34
 LIBS:power
 LIBS:device
@@
 Sheet 3 10
 Title "CPU circuit"
-Date "8 feb 2012"
+Date "11 feb 2012"
 Rev "0.01"
 Comp "diyefi.org"
@@
 NoConn ~ 11400 5450
 $Comp
-L +5V_MICRO #PWR014
+L +5V_MICRO #PWR012
 U 1 1 4F28F62D
 P 12550 3150
-F 0 "#PWR014" H 12550 3100 20  0001 C CNN
+F 0 "#PWR012" H 12550 3100 20  0001 C CNN
 F 1 "+5V_MICRO" H 12400 3200 30  0000 C CNN
 	1    12550 3150
@@
 $EndComp
 $Comp
-L GND #PWR015
+L GND #PWR013
 U 1 1 4F28F57C
 P 12550 3550
-F 0 "#PWR015" H 12550 3550 30  0001 C CNN
+F 0 "#PWR013" H 12550 3550 30  0001 C CNN
 F 1 "GND" H 12550 3480 30  0001 C CNN
 	1    12550 3550
@@
 $EndComp
 $Comp
-L GND #PWR016
+L GND #PWR014
 U 1 1 4F28B93D
 P 5700 7900
-F 0 "#PWR016" H 5700 7900 30  0001 C CNN
+F 0 "#PWR014" H 5700 7900 30  0001 C CNN
 F 1 "GND" H 5700 7830 30  0001 C CNN
 	1    5700 7900
@@
 P 3750 7600
 F 0 "C43" H 3800 7700 50  0000 L CNN
-F 1 ".1uF" H 3800 7500 50  0000 L CNN
+F 1 "0.1uF" H 3800 7500 50  0000 L CNN
 F 2 "C1V7" V 30  6700 60  0001 C CNN
 F 4 "newark,56K3664" V 30  6700 60  0001 C CNN "Field1"
@@
 $EndComp
 $Comp
-L +12V_SWITCHED #PWR017
+L +12V_SWITCHED #PWR015
 U 1 1 4F28B938
 P 3000 7400
-F 0 "#PWR017" H 3000 7350 20  0001 C CNN
+F 0 "#PWR015" H 3000 7350 20  0001 C CNN
 F 1 "+12V_SWITCHED" H 3000 7500 30  0000 C CNN
 	1    3000 7400
@@
 $EndComp
 $Comp
-L +5V_MICRO #PWR018
+L +5V_MICRO #PWR016
 U 1 1 4F28B937
 P 6100 7400
-F 0 "#PWR018" H 6100 7350 20  0001 C CNN
+F 0 "#PWR016" H 6100 7350 20  0001 C CNN
 F 1 "+5V_MICRO" H 6100 7500 30  0000 C CNN
 	1    6100 7400
@@
 Power symbols usage\n+12V_SWITCHED  come from igniton switch\n+5V_MICRO      come from CPU voltage reg         \n+5V_SWITCHED   come from secondary voltage reg\nLSGND          low side ground\nADCGND         sensor ground\nIGNGND         ignition ground
 $Comp
-L PWR_FLAG #FLG019
+L PWR_FLAG #FLG017
 U 1 1 4F28B936
 P 3400 7400
-F 0 "#FLG019" H 3400 7670 30  0001 C CNN
+F 0 "#FLG017" H 3400 7670 30  0001 C CNN
 F 1 "PWR_FLAG" H 3400 7630 30  0000 C CNN
 	1    3400 7400
@@
 $EndComp
 $Comp
-L +12V_SWITCHED #PWR020
+L +12V_SWITCHED #PWR018
 U 1 1 4F28B933
 P 3000 9300
-F 0 "#PWR020" H 3000 9250 20  0001 C CNN
+F 0 "#PWR018" H 3000 9250 20  0001 C CNN
 F 1 "+12V_SWITCHED" H 3000 9400 30  0000 C CNN
 	1    3000 9300
@@
 P 3750 9500
 F 0 "C48" H 3800 9600 50  0000 L CNN
-F 1 ".1uF" H 3800 9400 50  0000 L CNN
+F 1 "0.1uF" H 3800 9400 50  0000 L CNN
 F 2 "C1V7" V 30  8600 60  0001 C CNN
 F 4 "newark,56K3664" V 30  8600 60  0001 C CNN "Field1"
@@
 $EndComp
 $Comp
-L GND #PWR021
+L GND #PWR019
 U 1 1 4F28B92E
 P 5700 9800
-F 0 "#PWR021" H 5700 9800 30  0001 C CNN
+F 0 "#PWR019" H 5700 9800 30  0001 C CNN
 F 1 "GND" H 5700 9730 30  0001 C CNN
 	1    5700 9800
@@
 $EndComp
 $Comp
-L +5V_SWITCHED #PWR022
+L +5V_SWITCHED #PWR020
 U 1 1 4F28B92C
 P 6100 9300
-F 0 "#PWR022" H 6100 9250 20  0001 C CNN
+F 0 "#PWR020" H 6100 9250 20  0001 C CNN
 F 1 "+5V_SWITCHED" H 6100 9400 30  0000 C CNN
 	1    6100 9300
@@
 $EndComp
 $Comp
-L ADCGND #PWR023
+L ADCGND #PWR021
 U 1 1 4F28B92B
 P 5350 9800
-F 0 "#PWR023" H 5350 9800 40  0001 C CNN
+F 0 "#PWR021" H 5350 9800 40  0001 C CNN
 F 1 "ADCGND" H 5350 9730 40  0000 C CNN
 	1    5350 9800
@@
 $EndComp
 $Comp
-L GND #PWR024
+L GND #PWR022
 U 1 1 4F281768
 P 6750 5700
-F 0 "#PWR024" H 6750 5700 30  0001 C CNN
+F 0 "#PWR022" H 6750 5700 30  0001 C CNN
 F 1 "GND" H 6750 5630 30  0001 C CNN
 	1    6750 5700
@@
 $EndComp
 $Comp
-L +5V_MICRO #PWR025
+L +5V_MICRO #PWR023
 U 1 1 4F28154A
 P 8350 6750
-F 0 "#PWR025" H 8350 6700 20  0001 C CNN
+F 0 "#PWR023" H 8350 6700 20  0001 C CNN
 F 1 "+5V_MICRO" H 8350 6850 30  0000 C CNN
 	1    8350 6750
@@
 NoConn ~ 9350 7250
 $Comp
-L ADCGND #PWR026
+L ADCGND #PWR024
 U 1 1 4F26B6B4
 P 12400 4050
-F 0 "#PWR026" H 12400 4050 40  0001 C CNN
+F 0 "#PWR024" H 12400 4050 40  0001 C CNN
 F 1 "ADCGND" H 12400 3980 40  0000 C CNN
 	1    12400 4050
@@
 NoConn ~ 9350 7150
 $Comp
-L PWR_FLAG #FLG027
+L PWR_FLAG #FLG025
 U 1 1 4EF89402
 P 8650 2900
-F 0 "#FLG027" H 8650 3170 30  0001 C CNN
+F 0 "#FLG025" H 8650 3170 30  0001 C CNN
 F 1 "PWR_FLAG" H 8650 3130 30  0000 C CNN
 	1    8650 2900
@@
 $EndComp
 $Comp
-L +5V_SWITCHED #PWR028
+L +5V_SWITCHED #PWR026
 U 1 1 4EFBB324
 P 12400 3650
-F 0 "#PWR028" H 12400 3600 20  0001 C CNN
+F 0 "#PWR026" H 12400 3600 20  0001 C CNN
 F 1 "+5V_SWITCHED" H 12200 3700 30  0000 C CNN
 	1    12400 3650
@@
 NoConn ~ 11400 3750
 $Comp
-L +5V_MICRO #PWR029
+L +5V_MICRO #PWR027
 U 1 1 4EFB34CE
 P 6750 4500
-F 0 "#PWR029" H 6750 4450 20  0001 C CNN
+F 0 "#PWR027" H 6750 4450 20  0001 C CNN
 F 1 "+5V_MICRO" H 6750 4600 30  0000 C CNN
 	1    6750 4500
@@
 $EndComp
 $Comp
-L +5V_MICRO #PWR030
+L +5V_MICRO #PWR028
 U 1 1 4EFB34CB
 P 8300 4550
-F 0 "#PWR030" H 8300 4500 20  0001 C CNN
+F 0 "#PWR028" H 8300 4500 20  0001 C CNN
 F 1 "+5V_MICRO" H 8300 4650 30  0000 C CNN
 	1    8300 4550
@@
 $EndComp
 $Comp
-L +5V_MICRO #PWR031
+L +5V_MICRO #PWR029
 U 1 1 4EFB34C6
 P 9250 2050
-F 0 "#PWR031" H 9250 2000 20  0001 C CNN
+F 0 "#PWR029" H 9250 2000 20  0001 C CNN
 F 1 "+5V_MICRO" H 9250 2150 30  0000 C CNN
 	1    9250 2050
@@
 $EndComp
 $Comp
-L GND #PWR032
+L GND #PWR030
 U 1 1 4EF8A1A8
 P 8350 8300
-F 0 "#PWR032" H 8350 8300 30  0001 C CNN
+F 0 "#PWR030" H 8350 8300 30  0001 C CNN
 F 1 "GND" H 8350 8230 30  0001 C CNN
 	1    8350 8300
@@
 $EndComp
 $Comp
-L GND #PWR033
+L GND #PWR031
 U 1 1 4EF89421
 P 12400 2550
-F 0 "#PWR033" H 12400 2550 30  0001 C CNN
+F 0 "#PWR031" H 12400 2550 30  0001 C CNN
 F 1 "GND" H 12400 2480 30  0001 C CNN
 	1    12400 2550
@@
 $EndComp
 $Comp
-L GND #PWR034
+L GND #PWR032
 U 1 1 4EF89420
 P 12700 3050
-F 0 "#PWR034" H 12700 3050 30  0001 C CNN
+F 0 "#PWR032" H 12700 3050 30  0001 C CNN
 F 1 "GND" H 12700 2980 30  0001 C CNN
 	1    12700 3050
@@
 $EndComp
 $Comp
-L GND #PWR035
+L GND #PWR033
 U 1 1 4EF8941E
 P 8500 2600
-F 0 "#PWR035" H 8500 2600 30  0001 C CNN
+F 0 "#PWR033" H 8500 2600 30  0001 C CNN
 F 1 "GND" H 8500 2530 30  0001 C CNN
 	1    8500 2600
@@
 $EndComp
 $Comp
-L GND #PWR036
+L GND #PWR034
 U 1 1 4EF8941D
 P 8150 2950
-F 0 "#PWR036" H 8150 2950 30  0001 C CNN
+F 0 "#PWR034" H 8150 2950 30  0001 C CNN
 F 1 "GND" H 8150 2880 30  0001 C CNN
 	1    8150 2950
@@
 $EndComp
 $Comp
-L GND #PWR037
+L GND #PWR035
 U 1 1 4EF8941A
 P 11400 2350
-F 0 "#PWR037" H 11400 2350 30  0001 C CNN
+F 0 "#PWR035" H 11400 2350 30  0001 C CNN
 F 1 "GND" H 11400 2280 30  0001 C CNN
 	1    11400 2350
@@
 $EndComp
 $Comp
-L GND #PWR038
+L GND #PWR036
 U 1 1 4EF89415
 P 8300 4200
-F 0 "#PWR038" H 8300 4200 30  0001 C CNN
+F 0 "#PWR036" H 8300 4200 30  0001 C CNN
 F 1 "GND" H 8300 4130 30  0001 C CNN
 	1    8300 4200
@@
 PLL + CLK
 $Comp
-L GND #PWR039
+L GND #PWR037
 U 1 1 4EF89410
 P 4700 3500
-F 0 "#PWR039" H 4700 3500 30  0001 C CNN
+F 0 "#PWR037" H 4700 3500 30  0001 C CNN
 F 1 "GND" H 4700 3430 30  0001 C CNN
 	1    4700 3500
@@
 $EndComp
 $Comp
-L GND #PWR040
+L GND #PWR038
 U 1 1 4EF8940F
 P 5150 3200
-F 0 "#PWR040" H 5150 3200 30  0001 C CNN
+F 0 "#PWR038" H 5150 3200 30  0001 C CNN
 F 1 "GND" H 5150 3130 30  0001 C CNN
 	1    5150 3200
