File: design/Core Board.sch (KiCad schematic (older format))
At the start: 41 parts, among them K2 Bootldr, P1 BDM, U10 TLE4275, U2 MC9S12XDP512, U9 TLE4275, X1 CRYSTAL

Commit message: Heavily revise the ADC gnd, relayout gnd, power and ignition net
Parts:
- added R42: 0, symbol R
Connections:
- wire segments 118 -> 119
