File: design/Injectors.sch (KiCad schematic (older format))
At the start: 7 parts, among them Q9 vnp10n07

Commit message: revise schema according to Jaguar & Ravage project, eliminate as many errors as possible which were inherited from Puma board. Remove VSS interface, narrow band O2 interface, AC relay output, AC signal input. Make fuel injection configurable which can be batch fired or semi sequential fired
Parts:
- removed D34: DIODE, symbol DIODE
- removed W7: TEST, symbol TEST
- added D27, D29: 1N4148, symbol DIODE
- added D28: LED, symbol LED
- added P6: semi/batch, symbol CONN_2
- added Q1: vnp10n07, symbol MOS_N
- added R22: 2K4, symbol R
- added R23, R25, R26: 1K, symbol R
- added R27: 100K, symbol R
Connections:
- net labels added: PB1, PT4, PT5
- wire segments 14 -> 28
Other:
- note added: "My magic screw connector\nOpen = semi sequential injection\nClose = batch injection"
- note removed: "Drive 4 High-Z injectors for batch injection"
- moved on the sheet: D33, Q9, R66, R67, R68
