File: design/U_Dashboard Analogue Outputs.sch (KiCad schematic (older format))
At the start: 23 parts, among them Q1 vnp10n07, Q2 8050, Q3 MMBT3904LT1, U3 MC34151P

Commit message: revise schema according to Jaguar & Ravage project, eliminate as many errors as possible which were inherited from Puma board. Remove VSS interface, narrow band O2 interface, AC relay output, AC signal input. Make fuel injection configurable which can be batch fired or semi sequential fired
Parts:
- removed D12, D14: LED, symbol LED
- removed D13: DIODE, symbol DIODE
- removed Q1: vnp10n07, symbol MOS_N
- removed Q2: 8050, symbol NPN
- removed Q3: MMBT3904LT1, symbol NPN
- removed R20: 3K, symbol R
- removed R22, R29: 1K, symbol R
- removed R23, R28, R30: 100K, symbol R
- removed R25: 330, symbol R
- removed R27: 220R, symbol R
- removed SP1: SPEAKER, symbol SPEAKER
- removed W2: TEST, symbol TEST
- C25: value 0.1 -> 0.1uF
- C26: value 4.7 -> 4.7uF
- R24: value 100K -> ??
Connections:
- net labels added: PP5
- net labels removed: CHECK_ENGINE, PA2, PA3, PA4, PP1
- wire segments 51 -> 20
Other:
- note added: "Tachometer PWM output"
- note removed: "Warmup LED"
- note removed: "check engine lamp"
- note removed: "lose sync notify"
- note removed: "tachometer PWM output"
- moved on the sheet: C25, C26, C27, D11, R21, R24, U3
